File: 6809PC-6U.kicad_pcb (KiCad board)
At the start: 2 copper layers, 233.7 x 160 mm, 142 parts, among them K1 CONN_3, K2 CONN_3, K3 CONN_3, P1 C96ABC, P10 16.000Mhz, P11 CONN_4X2, P12 CONN_4, P13 1.8432 MHz CLK, P14 SERIAL, P15 CONN_5X2, P17 PARALLEL, P2 CONN_4X2, P3 CONN_1, P4 CONN_1, P5 CONN_1, P6 CONN_1, P7 CONN_1, P8 CONN_10X2, P9 POWER_SW, SW1 POWER, SW2 MOM CNCT, U10 74HCT14, U14 74LS138, U15 74LS245, U16 74LS245, U17 74LS245, U18 74LS245, U2 74LS244, U23 DS1233, U24 74LS163, U25 74LS240, U27 MC68B09, U28 74LS244, U29 74LS08, U3 74LS682, U30 74LS174, U31 74LS244, U32 74LS157, U33 74LS374, U34 74LS244, U35 SRAM-32K, U36 74LS245, U37 74LS138, U38 74LS257, U39 74LS257, U4 74LS86, U40 74LS244, U41 74LS244, U42 DS1302, U43 G65SC51P, U44 MAX232, U45 G65SC22P, U46 G65SC22P, U5 74LS02, U6 74LS00, U7 74LS32, U8 SRAM_512K, U9 29F040, X1 RTC_OSC

Commit message: Schematic in progress
Parts:
- removed the JP3 at (186.7, 199.4)
- removed the P1 at (243.8, 196.8)
- removed the R1 at (146.1, 120.7)
- removed the R5 at (186.7, 196.8)
- removed the R6 at (186.7, 194.3)
- removed the U29 at (158.8, 146.1)
- removed the U42 at (109.2, 119.4)
- removed XK1: CONN_3X2, PIN_ARRAY_3x2
- removed XK2: CONN_3, PIN_ARRAY_3X1
- added C56: 0.1 uF, Capacitor_THT:C_Disc_D5.0mm_W2.5mm_P5.00mm, F.Cu at (347.4, 170.2)
- added C57: 0.01 uF, Capacitor_THT:C_Disc_D5.0mm_W2.5mm_P5.00mm, F.Cu at (391.4, 170.2)
- added C59: 15pf, Capacitor_THT:C_Disc_D5.0mm_W2.5mm_P5.00mm, F.Cu at (450.3, 146.2)
- added C60: 15pf, Capacitor_THT:C_Disc_D5.0mm_W2.5mm_P5.00mm, F.Cu at (450.3, 150.3)
- added C67: 0.1µF, Capacitor_THT:C_Disc_D5.0mm_W2.5mm_P5.00mm, F.Cu at (368.6, 153.5)
- added C68: 10µF, Capacitor_THT:CP_Radial_D5.0mm_P2.50mm, F.Cu at (369.1, 158.8)
- added D3: D, Diode_THT:D_DO-41_SOD81_P10.16mm_Horizontal, F.Cu at (450.6, 137.8)
- added D4: D, Diode_THT:D_DO-41_SOD81_P10.16mm_Horizontal, F.Cu at (450.6, 142.1)
- added D5: 1N4001, Diode_THT:D_DO-41_SOD81_P10.16mm_Horizontal, F.Cu at (383.0, 156.7)
- added D6: 1N4001, Diode_THT:D_DO-41_SOD81_P10.16mm_Horizontal, F.Cu at (383.0, 161.0)
- added J1: IRQ Selection, Connector_PinHeader_2.54mm:PinHeader_2x06_P2.54mm_Vertical, F.Cu at (336.4, 58.2)
- added J10: AUDIO OUT, Connector_PinHeader_2.54mm:PinHeader_1x02_P2.54mm_Horizontal, F.Cu at (408.5, 97.4)
- added J11: TTL SERIAL 0, Connector_PinHeader_2.54mm:PinHeader_1x06_P2.54mm_Horizontal, F.Cu at (396.7, 104.6)
- added J12: TTL SER 0 PWR, Connector_PinHeader_2.54mm:PinHeader_1x02_P2.54mm_Vertical, F.Cu at (369.4, 146.6)
- added J13: TTL SERIAL 1, Connector_PinHeader_2.54mm:PinHeader_1x06_P2.54mm_Horizontal, F.Cu at (410.1, 104.6)
- added J14: TTL SER 1 PWR, Connector_PinHeader_2.54mm:PinHeader_1x02_P2.54mm_Vertical, F.Cu at (374.0, 146.6)
- added J2: Bus_ISA_8bit, Custom:BUSPC_HOST, F.Cu at (66.2, 91.2)
- added J3: TTL SERIAL CONSOLE, Connector_PinHeader_2.54mm:PinHeader_1x06_P2.54mm_Horizontal, F.Cu at (372.1, 170.5)
- added J4: TTL CONSOLE PWR, Connector_PinHeader_2.54mm:PinHeader_1x02_P2.54mm_Vertical, F.Cu at (385.5, 170.5)
- added J5: KEYBOARD AND MOUSE, Connector_PinHeader_2.54mm:PinHeader_2x05_P2.54mm_Horizontal, F.Cu at (404.9, 152.4)
- added J6: VGA, Connector_Dsub:DSUB-15-HD_Female_Horizontal_P2.29x1.98mm_EdgePinOffset3.03mm_Housed_MountingHolesOffset4.94mm, F.Cu at (354.9, 147.4)
- added J7: VGA, Connector_PinHeader_2.54mm:PinHeader_1x07_P2.54mm_Horizontal, F.Cu at (408.5, 77.5)
- added J8: Keyboard, Custom:PS2_DIN, F.Cu at (411.0, 130.4)
- added J9: Mouse, Custom:PS2_DIN, F.Cu at (411.0, 144.4)
- added JP4: JUMPER, Connector_PinHeader_2.54mm:PinHeader_1x02_P2.54mm_Vertical, F.Cu at (446.5, 172.7)
- added P9: 14.31818 MHz CLK, Package_DIP:DIP-14_W7.62mm_Socket_LongPads, F.Cu at (336.2, 170.3)
- added R10: 390Ω, Resistor_THT:R_Axial_DIN0207_L6.3mm_D2.5mm_P7.62mm_Horizontal, F.Cu at (382.7, 132.3)
- added R11: 820Ω, Resistor_THT:R_Axial_DIN0207_L6.3mm_D2.5mm_P7.62mm_Horizontal, F.Cu at (382.7, 136.4)
- added R12: 390Ω, Resistor_THT:R_Axial_DIN0207_L6.3mm_D2.5mm_P7.62mm_Horizontal, F.Cu at (382.7, 140.4)
- added R13: 820Ω, Resistor_THT:R_Axial_DIN0207_L6.3mm_D2.5mm_P7.62mm_Horizontal, F.Cu at (382.7, 144.5)
- added R14: 120Ω, Resistor_THT:R_Axial_DIN0207_L6.3mm_D2.5mm_P7.62mm_Horizontal, F.Cu at (382.7, 148.5)
- added R15: 120Ω, Resistor_THT:R_Axial_DIN0207_L6.3mm_D2.5mm_P7.62mm_Horizontal, F.Cu at (382.7, 152.6)
- added R16: 2.2KΩ, Resistor_THT:R_Axial_DIN0207_L6.3mm_D2.5mm_P7.62mm_Horizontal, F.Cu at (393.4, 124.2)
- added R17: 1KΩ, Resistor_THT:R_Axial_DIN0207_L6.3mm_D2.5mm_P7.62mm_Horizontal, F.Cu at (393.4, 128.3)
- added R18: 2.2KΩ, Resistor_THT:R_Axial_DIN0207_L6.3mm_D2.5mm_P7.62mm_Horizontal, F.Cu at (393.4, 132.3)
- added R19: 1KΩ, Resistor_THT:R_Axial_DIN0207_L6.3mm_D2.5mm_P7.62mm_Horizontal, F.Cu at (393.4, 136.4)
- added R20: 120Ω, Resistor_THT:R_Axial_DIN0207_L6.3mm_D2.5mm_P7.62mm_Horizontal, F.Cu at (393.4, 140.4)
- added R21: 120Ω, Resistor_THT:R_Axial_DIN0207_L6.3mm_D2.5mm_P7.62mm_Horizontal, F.Cu at (393.4, 144.5)
- added R22: 270Ω, Resistor_THT:R_Axial_DIN0207_L6.3mm_D2.5mm_P7.62mm_Horizontal, F.Cu at (393.4, 148.5)
- added R23: 150Ω, Resistor_THT:R_Axial_DIN0207_L6.3mm_D2.5mm_P7.62mm_Horizontal, F.Cu at (393.4, 152.6)
- added R24: 22K, Resistor_THT:R_Axial_DIN0207_L6.3mm_D2.5mm_P7.62mm_Horizontal, F.Cu at (445.7, 164.3)
- added R25: 22K, Resistor_THT:R_Axial_DIN0207_L6.3mm_D2.5mm_P7.62mm_Horizontal, F.Cu at (445.7, 168.3)
- added R8: 390Ω, Resistor_THT:R_Axial_DIN0207_L6.3mm_D2.5mm_P7.62mm_Horizontal, F.Cu at (382.7, 124.2)
- added R9: 820Ω, Resistor_THT:R_Axial_DIN0207_L6.3mm_D2.5mm_P7.62mm_Horizontal, F.Cu at (382.7, 128.3)
- added RN1: 1KΩ, Resistor_THT:R_Array_SIP9, F.Cu at (336.3, 164.0)
- added U1: 74LS04, Package_DIP:DIP-14_W7.62mm_Socket_LongPads, F.Cu at (358.1, 170.3)
- added U10: 74LS32, Package_DIP:DIP-14_W7.62mm_Socket_LongPads, F.Cu at (425.3, 77.3)
- added U11: 74LS32, Package_DIP:DIP-14_W7.62mm_Socket_LongPads, F.Cu at (437.0, 77.3)
- added U12: 74LS32, Package_DIP:DIP-14_W7.62mm_Socket_LongPads, F.Cu at (448.8, 77.3)
- added U13: 74LS07, Package_DIP:DIP-14_W7.62mm_Socket_LongPads, F.Cu at (460.5, 77.3)
- added U14: 74LS07, Package_DIP:DIP-14_W7.62mm_Socket_LongPads, F.Cu at (425.3, 96.8)
- added U15: 74LS08, Package_DIP:DIP-14_W7.62mm_Socket_LongPads, F.Cu at (437.0, 96.8)
- added U16: 74LS32, Package_DIP:DIP-14_W7.62mm_Socket_LongPads, F.Cu at (448.8, 96.8)
- added U17: 74LS14, Package_DIP:DIP-14_W7.62mm_Socket_LongPads, F.Cu at (460.5, 96.8)
- added U18: 74LS06, Package_DIP:DIP-14_W7.62mm_Socket_LongPads, F.Cu at (425.3, 116.3)
- added U20: 74LS04, Package_DIP:DIP-14_W7.62mm_Socket_LongPads, F.Cu at (437.0, 116.3)
- added U21: 74LS00, Package_DIP:DIP-14_W7.62mm_Socket_LongPads, F.Cu at (448.8, 116.3)
- added U22: 74LS74, Package_DIP:DIP-14_W7.62mm_Socket_LongPads, F.Cu at (460.5, 116.3)
- added U31: 74LS245, Package_DIP:DIP-20_W7.62mm_Socket_LongPads, F.Cu at (425.3, 137.8)
- added U46: ~, Package_DIP:DIP-18_W7.62mm_Socket_LongPads, F.Cu at (439.0, 137.8)
- added U49: 74HC595, Package_DIP:DIP-16_W7.62mm_Socket_LongPads, F.Cu at (336.2, 124.3)
- added U50: 74HC165, Package_DIP:DIP-16_W7.62mm_Socket_LongPads, F.Cu at (347.9, 124.3)
- added U51: 74HC595, Package_DIP:DIP-16_W7.62mm_Socket_LongPads, F.Cu at (359.7, 124.3)
- added U52: 74HC165, Package_DIP:DIP-16_W7.62mm_Socket_LongPads, F.Cu at (371.4, 124.3)
- added U53: ESP32_MODULE, Custom:ESP32_Module, F.Cu at (348.5, 76.0)
- added U54: ESP32_MODULE, Custom:ESP32_Module, F.Cu at (378.6, 76.0)
- added U55: 74LS244, Package_DIP:DIP-20_W7.62mm_Socket_LongPads, F.Cu at (396.5, 77.3)
- C1, C2, C28, C3, C35, C4: footprint C1V5 -> Capacitor_THT:CP_Radial_D5.0mm_P2.50mm
- C10, C11, C12, C13, C14, C15, C16, C17, C18, C19, C20, C21, C22, C23, C24, C25, C26, C27, C29, C30, C31, C32, C33, C34, C36, C37, C38, C39, C40, C41, C42, C43, C44, C45, C46, C47, C48, C49, C5, C50, C51, C52, C53, C54, C55, C6, C7, C8, C9: footprint C2 -> Capacitor_THT:C_Disc_D5.0mm_W2.5mm_P5.00mm
- C58: renamed from C57; footprint C2 -> Capacitor_THT:C_Disc_D5.0mm_W2.5mm_P5.00mm
- C61: renamed from C58; footprint C1V5 -> Capacitor_THT:CP_Radial_D5.0mm_P2.50mm
- C62: renamed from C59; footprint C2 -> Capacitor_THT:C_Disc_D5.0mm_W2.5mm_P5.00mm
- C63: renamed from C60; footprint C1V5 -> Capacitor_THT:CP_Radial_D5.0mm_P2.50mm
- C64: renamed from C61; footprint C1V5 -> Capacitor_THT:CP_Radial_D5.0mm_P2.50mm
- C65: renamed from C62; footprint C1V5 -> Capacitor_THT:CP_Radial_D5.0mm_P2.50mm
- C66: renamed from C63; footprint C1V5 -> Capacitor_THT:CP_Radial_D5.0mm_P2.50mm
- D1, D2: footprint D3 -> Diode_THT:D_DO-41_SOD81_P10.16mm_Horizontal
- JP1, JP2, JP5: footprint PIN_ARRAY_2X1 -> Connector_PinHeader_2.54mm:PinHeader_1x02_P2.54mm_Vertical
- JP3: renamed from JP4; footprint PIN_ARRAY_2X1 -> Connector_PinHeader_2.54mm:PinHeader_1x02_P2.54mm_Vertical
- K1, K2, K3: footprint PIN_ARRAY_3X1 -> Connector_PinHeader_2.54mm:PinHeader_1x03_P2.54mm_Vertical
- P1: renamed from P2; footprint PIN_ARRAY_4x2 -> Connector_PinHeader_2.54mm:PinHeader_2x04_P2.54mm_Vertical
- P10, P13, U4, U5, U6, U7: footprint DIP-14__300 -> Package_DIP:DIP-14_W7.62mm_Socket_LongPads
- P11: footprint PIN_ARRAY_4x2 -> Connector_PinHeader_2.54mm:PinHeader_2x04_P2.54mm_Vertical
- P12: footprint PIN_ARRAY_4x1 -> Connector_PinHeader_2.54mm:PinHeader_1x04_P2.54mm_Vertical
- P14: footprint PIN_ARRAY_5x2 -> Connector_PinHeader_2.54mm:PinHeader_2x05_P2.54mm_Vertical
- P15: value CONN_5X2 -> CONN_8X2; footprint PIN_ARRAY_5x2 -> Connector_PinHeader_2.54mm:PinHeader_2x08_P2.54mm_Vertical
- P16: renamed from P17; footprint PIN_ARRAY_13x2 -> Connector_PinHeader_2.54mm:PinHeader_2x13_P2.54mm_Vertical
- P2: renamed from P3; footprint 1pin -> MountingHole:MountingHole_2.7mm_M2.5_Pad_TopBottom
- P3: renamed from P4; footprint 1pin -> MountingHole:MountingHole_2.7mm_M2.5_Pad_TopBottom
- P4: renamed from P5; footprint 1pin -> MountingHole:MountingHole_2.7mm_M2.5_Pad_TopBottom
- P5: renamed from P6; footprint 1pin -> MountingHole:MountingHole_2.7mm_M2.5_Pad_TopBottom
- P6: renamed from P7; footprint 1pin -> MountingHole:MountingHole_2.7mm_M2.5_Pad_TopBottom
- P7: renamed from P8; footprint ATX_NON_90DEG -> Custom:ATXConnector
- P8: renamed from P9; footprint PIN_ARRAY_2X1 -> Connector_PinHeader_2.54mm:PinHeader_1x02_P2.54mm_Vertical
- R1: renamed from R2; footprint R3 -> Resistor_THT:R_Axial_DIN0207_L6.3mm_D2.5mm_P7.62mm_Horizontal
- R2: renamed from R3; footprint R3 -> Resistor_THT:R_Axial_DIN0207_L6.3mm_D2.5mm_P7.62mm_Horizontal
- R3: renamed from R4; footprint R3 -> Resistor_THT:R_Axial_DIN0207_L6.3mm_D2.5mm_P7.62mm_Horizontal
- R4: renamed from R7; footprint R3 -> Resistor_THT:R_Axial_DIN0207_L6.3mm_D2.5mm_P7.62mm_Horizontal
- R5: renamed from R8; footprint R3 -> Resistor_THT:R_Axial_DIN0207_L6.3mm_D2.5mm_P7.62mm_Horizontal
- R6: renamed from R9; footprint R3 -> Resistor_THT:R_Axial_DIN0207_L6.3mm_D2.5mm_P7.62mm_Horizontal
- R7: renamed from R10; footprint R3 -> Resistor_THT:R_Axial_DIN0207_L6.3mm_D2.5mm_P7.62mm_Horizontal
- SW1, SW2: footprint SW_PUSH_SMALL -> Button_Switch_THT:SW_Tactile_Straight_KSL0Axx1LFTR
- U19: renamed from U10; footprint DIP-14__300 -> Package_DIP:DIP-14_W7.62mm_Socket_LongPads
- U2, U3: footprint DIP-20__300 -> Package_DIP:DIP-20_W7.62mm_Socket_LongPads
- U23: renamed from U14; footprint DIP-16__300 -> Package_DIP:DIP-16_W7.62mm_Socket_LongPads
- U24: renamed from U15; footprint DIP-20__300 -> Package_DIP:DIP-20_W7.62mm_Socket_LongPads
- U25: renamed from U16; footprint DIP-20__300 -> Package_DIP:DIP-20_W7.62mm_Socket_LongPads
- U26: renamed from U17; footprint DIP-20__300 -> Package_DIP:DIP-20_W7.62mm_Socket_LongPads
- U27: renamed from U18; footprint DIP-20__300 -> Package_DIP:DIP-20_W7.62mm_Socket_LongPads
- U29: renamed from U24; footprint DIP-16__300 -> Package_DIP:DIP-16_W7.62mm_Socket_LongPads
- U30: renamed from U25; footprint DIP-20__300 -> Package_DIP:DIP-20_W7.62mm_Socket_LongPads
- U32: renamed from U27; footprint Package_DIP:DIP-40_W15.24mm -> Package_DIP:DIP-40_W15.24mm_Socket_LongPads
- U33: renamed from U28; footprint DIP-20__300 -> Package_DIP:DIP-20_W7.62mm_Socket_LongPads
- U34: renamed from U30; footprint DIP-16__300 -> Package_DIP:DIP-16_W7.62mm_Socket_LongPads
- U35: renamed from U31; footprint DIP-20__300 -> Package_DIP:DIP-20_W7.62mm_Socket_LongPads
- U36: renamed from U32; footprint DIP-16__300 -> Package_DIP:DIP-16_W7.62mm_Socket_LongPads
- U37: renamed from U33; footprint DIP-20__300 -> Package_DIP:DIP-20_W7.62mm_Socket_LongPads
- U38: renamed from U34; footprint DIP-20__300 -> Package_DIP:DIP-20_W7.62mm_Socket_LongPads
- U39: renamed from U35; footprint Package_DIP:DIP-28_W15.24mm -> Package_DIP:DIP-28_W7.62mm_Socket_LongPads
- U40: renamed from U36; footprint DIP-20__300 -> Package_DIP:DIP-20_W7.62mm_Socket_LongPads
- U41: renamed from U37; footprint DIP-16__300 -> Package_DIP:DIP-16_W7.62mm_Socket_LongPads
- U42: renamed from U38; footprint DIP-16__300 -> Package_DIP:DIP-16_W7.62mm_Socket_LongPads
- U43: renamed from U39; footprint DIP-16__300 -> Package_DIP:DIP-16_W7.62mm_Socket_LongPads
- U44: renamed from U40; footprint DIP-20__300 -> Package_DIP:DIP-20_W7.62mm_Socket_LongPads
- U45: renamed from U41; footprint DIP-20__300 -> Package_DIP:DIP-20_W7.62mm_Socket_LongPads
- U47: renamed from U43; footprint DIP-28__600 -> Package_DIP:DIP-28_W15.24mm_Socket_LongPads
- U48: renamed from U44; footprint DIP-16__300 -> Package_DIP:DIP-16_W7.62mm_Socket_LongPads
- U56: renamed from U45; footprint DIP-40__600 -> Package_DIP:DIP-40_W15.24mm_Socket_LongPads
- U57: renamed from U46; footprint DIP-40__600 -> Package_DIP:DIP-40_W15.24mm_Socket_LongPads
- U8: footprint Package_DIP:DIP-32_W15.24mm -> Package_DIP:DIP-32_W15.24mm_Socket_LongPads
- U9: footprint DIP-32__600 -> Package_DIP:DIP-32_W15.24mm_Socket_LongPads
- X1: footprint C1 -> Crystal:Crystal_DS10_D1.0mm_L4.3mm_Horizontal
- moved C18 454.3 mm to (564.4, 56.9)
- moved C22 454.3 mm to (572.0, 102.6)
- moved C31 454.3 mm to (646.9, 116.6)
- moved C32 454.3 mm to (612.6, 116.6)
- moved C33 454.3 mm to (556.8, 101.3)
- moved C36 454.3 mm to (555.5, 116.6)
- moved C37 454.3 mm to (602.5, 56.9)
- moved C40 454.3 mm to (525.0, 56.9)
- moved C41 454.3 mm to (589.8, 116.6)
- moved C45 454.3 mm to (532.6, 116.6)
- moved C53 454.3 mm to (621.5, 56.9)
- moved C55 454.3 mm to (635.5, 116.6)
- moved C58 454.3 mm to (662.2, 116.6)
- moved C6 454.3 mm to (583.4, 56.9)
- moved C61 454.3 mm to (605.0, 44.2)
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- renumbered U23 to U28
Connections:
- K1 pad 2: Net-(K1-Pin_2) -> PULLUP2
- P15 pad 1: /ACIA/RTS_TTL -> VCC
- P15 pad 10: /ACIA/DTR -> PD4
- P15 pad 2: VCC -> PD0
- P15 pad 3: /ACIA/TXD_TTL -> /VIAS/CA1
- P15 pad 4: /ACIA/RXCLK -> PD1
- P15 pad 5: /ACIA/CTS_TTL -> /VIAS/CA2
- P15 pad 6: /ACIA/DSR -> PD2
- P15 pad 7: /ACIA/RXD_TTL -> /VIAS/CB1
- P15 pad 8: /ACIA/DCD -> PD3
- P15 pad 9: GND -> /VIAS/CB2
- P7 pad 16: unconnected-(P8-Pin_16-Pad16) -> -5V
- P7 pad 19: unconnected-(P8-Pin_19-Pad19) -> +12V
- P7 pad 4: unconnected-(P8-Pin_4-Pad4) -> -12V
- RR1 pad 3: SD_SEL -> PULLUP1
- RR1 pad 4: B_/WAIT -> PULLUP2
- RR1 pad 5: /PG -> PULLUP3
- RR1 pad 7: B_/M1 -> PULLUP4
- RR2 pad 4: /SO -> unconnected-(RR2-R3-Pad4)
- U30 pad 12: B_DT/R -> unconnected-(U30-O3a-Pad12)
- U30 pad 8: R/W -> unconnected-(U30-I3a-Pad8)
- U32 pad 33: /BUSRQ -> unconnected-(U32-~{DMA/BREQ}-Pad33)
- U33 pad 11: /BUSAK -> unconnected-(U33-I0b-Pad11)
- U33 pad 13: B_/BUSRQ -> unconnected-(U33-I1b-Pad13)
- U33 pad 2: Net-(U28-I0a) -> Net-(U33-I0a)
- U33 pad 7: /BUSRQ -> unconnected-(U33-O1b-Pad7)
- U33 pad 9: B_/BUSAK -> unconnected-(U33-O0b-Pad9)
- U43 pad 16: unconnected-(U39-VCC-Pad16) -> VCC
- U47 pad 5: /ACIA/RXCLK -> unconnected-(U47-RxC-Pad5)
- U5 pad 1: Net-(XK2-Pin_3) -> Net-(U33-I0a)
- U5 pad 3: Net-(U5-Pad3) -> CPU_Q
- U57 pad 18: /VIAS/CD1 -> CD1
- U7 pad 11: unconnected-(U7-Pad11) -> SMEMW
- U7 pad 12: unconnected-(U7-Pad12) -> B_/IORQ
- U7 pad 13: unconnected-(U7-Pad13) -> B_/WR
- U9 pad 31: Net-(K1-Pin_2) -> PULLUP2
Routing:
- net (no net): track 7222.6 -> 0.00 mm, vias 45 -> 0
- net GND: track 2129.1 -> 0.00 mm, vias 1 -> 0
- net +5V: track 1301.0 -> 0.00 mm
- net mD7: track 554.9 -> 0.00 mm, vias 7 -> 0
- net mD2: track 537.2 -> 0.00 mm, vias 2 -> 0
- net mD6: track 528.1 -> 0.00 mm, vias 3 -> 0
- net mD1: track 525.1 -> 0.00 mm, vias 1 -> 0
- net mD3: track 518.8 -> 0.00 mm, vias 2 -> 0
- net mD4: track 506.6 -> 0.00 mm, vias 2 -> 0
- net mD0: track 491.2 -> 0.00 mm, vias 2 -> 0
- net mD5: track 475.9 -> 0.00 mm, vias 2 -> 0
- net /RESET: track 472.0 -> 0.00 mm, vias 5 -> 0
- net +3V3: track 456.9 -> 0.00 mm, vias 2 -> 0
- net mA0: track 450.2 -> 0.00 mm, vias 5 -> 0
- net mA17: track 432.6 -> 0.00 mm, vias 4 -> 0
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- removed copper zone on F.Cu, net (none)

Commit message: PCB in progress
Parts:
- added J1: IRQ Selection, Custom:STD_DDW_PINHEAD_V_2x06, F.Cu at (83.9, 148.5)
- added J10: Bus_ISA_8bit, Custom:BUSPC_HOST, F.Cu at (156.2, 117.7)
- added J2: IRQ Selection, Custom:STD_DDW_PINHEAD_V_2x06, F.Cu at (104.6, 148.5)
- added J3: Bus_ISA_8bit, Custom:BUSPC_HOST, F.Cu at (74.9, 117.7)
- added J4: Bus_ISA_8bit, Custom:BUSPC_HOST, F.Cu at (95.2, 117.7)
- added J5: IRQ Selection, Custom:STD_DDW_PINHEAD_V_2x06, F.Cu at (124.9, 148.3)
- added J6: Bus_ISA_8bit, Custom:BUSPC_HOST, F.Cu at (115.5, 117.7)
- added J9: IRQ Selection, Custom:STD_DDW_PINHEAD_V_2x06, F.Cu at (165.3, 148.4)
- added P10: CONN_1, MountingHole:MountingHole_3.2mm_M3_Pad_TopBottom, F.Cu at (306.5, 293.7)
- added P21: CONN_1, MountingHole:MountingHole_3.2mm_M3_Pad_TopBottom, F.Cu at (306.5, 89.2)
- added P22: CONN_1, MountingHole:MountingHole_3.2mm_M3_Pad_TopBottom, F.Cu at (83.0, 221.3)
- added P23: CONN_1, MountingHole:MountingHole_3.2mm_M3_Pad_TopBottom, F.Cu at (103.3, 221.3)
- added P4: CONN_1, MountingHole:MountingHole_3.2mm_M3_Pad_TopBottom, F.Cu at (149.0, 293.7)
- added P8: CONN_1, MountingHole:MountingHole_3.2mm_M3_Pad_TopBottom, F.Cu at (149.0, 221.3)
- added P9: CONN_1, MountingHole:MountingHole_3.2mm_M3_Pad_TopBottom, F.Cu at (306.5, 221.3)
- added U24: 74LS138, Custom:STD_DDW_DIP16, F.Cu at (206.5, 115.9)
- C1, C2, C28, C3, C35, C4, C61, C63, C64, C65, C66, C68: footprint Capacitor_THT:CP_Radial_D5.0mm_P2.50mm -> Custom:STD_DDW_PCAP
- C10, C11, C12, C13, C14, C15, C16, C17, C18, C19, C20, C21, C22, C23, C24, C25, C26, C27, C29, C30, C31, C32, C33, C34, C36, C37, C38, C39, C40, C41, C42, C43, C44, C45, C46, C47, C48, C49, C5, C50, C51, C52, C53, C54, C55, C56, C57, C58, C59, C6, C60, C62, C67, C7, C8, C9: footprint Capacitor_THT:C_Disc_D5.0mm_W2.5mm_P5.00mm -> Custom:STD_DDW_CAP
- D1, D2, D3, D4, D5, D6: footprint Diode_THT:D_DO-41_SOD81_P10.16mm_Horizontal -> Custom:STD_DDW_DIODE
- J11: renamed from J3; footprint Connector_PinHeader_2.54mm:PinHeader_1x06_P2.54mm_Horizontal -> Custom:STD_DDW_PINHEAD_V_1x06
- J12: renamed from J4; footprint Connector_PinHeader_2.54mm:PinHeader_1x02_P2.54mm_Vertical -> Custom:STD_DDW_PINHEAD_V_1x02
- J13: renamed from J5; footprint Connector_PinHeader_2.54mm:PinHeader_2x05_P2.54mm_Horizontal -> Custom:STD_DDW_PINHEAD_V_2x05
- J14: renamed from J6; footprint Connector_Dsub:DSUB-15-HD_Female_Horizontal_P2.29x1.98mm_EdgePinOffset3.03mm_Housed_MountingHolesOffset4.94mm -> Custom:STD_DDW_VGA
- J15: renamed from J7; footprint Connector_PinHeader_2.54mm:PinHeader_1x07_P2.54mm_Horizontal -> Custom:STD_DDW_PINHEAD_V_1x07
- J18: renamed from J10; footprint Connector_PinHeader_2.54mm:PinHeader_1x02_P2.54mm_Horizontal -> Custom:STD_DDW_PINHEAD_V_1x02
- J19: renamed from J11; footprint Connector_PinHeader_2.54mm:PinHeader_1x06_P2.54mm_Horizontal -> Custom:STD_DDW_PINHEAD_V_1x06
- J20: renamed from J12; footprint Connector_PinHeader_2.54mm:PinHeader_1x02_P2.54mm_Vertical -> Custom:STD_DDW_PINHEAD_V_1x02
- J21: renamed from J13; footprint Connector_PinHeader_2.54mm:PinHeader_1x06_P2.54mm_Horizontal -> Custom:STD_DDW_PINHEAD_V_1x06
- J22: renamed from J14; footprint Connector_PinHeader_2.54mm:PinHeader_1x02_P2.54mm_Vertical -> Custom:STD_DDW_PINHEAD_V_1x02
- J7: renamed from J1; footprint Connector_PinHeader_2.54mm:PinHeader_2x06_P2.54mm_Vertical -> Custom:STD_DDW_PINHEAD_V_2x06
- JP1: value JUMPER -> RESET; footprint Connector_PinHeader_2.54mm:PinHeader_1x02_P2.54mm_Vertical -> Custom:STD_DDW_PINHEAD_V_1x02
- JP2: value JUMPER -> CPU XTAL; footprint Connector_PinHeader_2.54mm:PinHeader_1x02_P2.54mm_Vertical -> Custom:STD_DDW_PINHEAD_V_1x02
- JP3: value JUMPER -> CTS; footprint Connector_PinHeader_2.54mm:PinHeader_1x02_P2.54mm_Vertical -> Custom:STD_DDW_PINHEAD_V_1x02
- JP4: value JUMPER -> OPT1; footprint Connector_PinHeader_2.54mm:PinHeader_1x02_P2.54mm_Vertical -> Custom:STD_DDW_PINHEAD_V_1x02
- JP5: value JUMPER -> OPT2; footprint Connector_PinHeader_2.54mm:PinHeader_1x02_P2.54mm_Vertical -> Custom:STD_DDW_PINHEAD_V_1x02
- K1: value CONN_3 -> EPROM/FLASH; footprint Connector_PinHeader_2.54mm:PinHeader_1x03_P2.54mm_Vertical -> Custom:STD_DDW_PINHEAD_V_1x03
- K2: value CONN_3 -> MMU DISABLE; footprint Connector_PinHeader_2.54mm:PinHeader_1x03_P2.54mm_Vertical -> Custom:STD_DDW_PINHEAD_V_1x03
- K3: value CONN_3 -> P Port Power; footprint Connector_PinHeader_2.54mm:PinHeader_1x03_P2.54mm_Vertical -> Custom:STD_DDW_PINHEAD_V_1x03
- P1: value CONN_4X2 -> SHADOW ADDR; footprint Connector_PinHeader_2.54mm:PinHeader_2x04_P2.54mm_Vertical -> Custom:STD_DDW_PINHEAD_V_2x04
- P12: renamed from P8; footprint Connector_PinHeader_2.54mm:PinHeader_1x02_P2.54mm_Vertical -> Custom:STD_DDW_PINHEAD_V_1x02
- P13: renamed from P9; footprint Package_DIP:DIP-14_W7.62mm_Socket_LongPads -> Custom:STD_DDW_DIP14
- P14: renamed from P10; footprint Package_DIP:DIP-14_W7.62mm_Socket_LongPads -> Custom:STD_DDW_DIP14
- P15: renamed from P11; value CONN_4X2 -> CPU CLOCK SPEED; footprint Connector_PinHeader_2.54mm:PinHeader_2x04_P2.54mm_Vertical -> Custom:STD_DDW_PINHEAD_V_2x04
- P16: renamed from P12; footprint Connector_PinHeader_2.54mm:PinHeader_1x04_P2.54mm_Vertical -> Custom:STD_DDW_PINHEAD_V_1x04
- P17: renamed from P13; footprint Package_DIP:DIP-14_W7.62mm_Socket_LongPads -> Custom:STD_DDW_DIP14
- P18: renamed from P14; footprint Connector_PinHeader_2.54mm:PinHeader_2x05_P2.54mm_Vertical -> Custom:STD_DDW_PINHEAD_V_2x05
- P19: renamed from P15; value CONN_8X2 -> VIA OUTPUT; footprint Connector_PinHeader_2.54mm:PinHeader_2x08_P2.54mm_Vertical -> Custom:STD_DDW_PINHEAD_V_2x08
- P2, P3: footprint MountingHole:MountingHole_2.7mm_M2.5_Pad_TopBottom -> MountingHole:MountingHole_3.2mm_M3_Pad_TopBottom
- P20: renamed from P16; footprint Connector_PinHeader_2.54mm:PinHeader_2x13_P2.54mm_Vertical -> Custom:STD_DDW_PINHEAD_V_2x13
- P5: renamed from P4; footprint MountingHole:MountingHole_2.7mm_M2.5_Pad_TopBottom -> MountingHole:MountingHole_3.2mm_M3_Pad_TopBottom
- P6: renamed from P5; footprint MountingHole:MountingHole_2.7mm_M2.5_Pad_TopBottom -> MountingHole:MountingHole_3.2mm_M3_Pad_TopBottom
- P7: renamed from P6; footprint MountingHole:MountingHole_2.7mm_M2.5_Pad_TopBottom -> MountingHole:MountingHole_3.2mm_M3_Pad_TopBottom
- R1, R10, R11, R12, R13, R14, R15, R16, R17, R18, R19, R2, R20, R21, R22, R23, R24, R25, R3, R4, R5, R6, R7, R8, R9: footprint Resistor_THT:R_Axial_DIN0207_L6.3mm_D2.5mm_P7.62mm_Horizontal -> Custom:STD_DDW_RESISTOR
- RN1: footprint Resistor_THT:R_Array_SIP9 -> Custom:STD_DDW_SIP9
- RR1, RR2: footprint Resistor_THT:R_Array_SIP10 -> Custom:STD_DDW_SIP10
- SW1, SW2: footprint Button_Switch_THT:SW_Tactile_Straight_KSL0Axx1LFTR -> Custom:STD_DDW_TACTSW
- U1, U10, U11, U12, U13, U14, U15, U16, U17, U18, U19, U20, U21, U22, U4, U5, U6, U7: footprint Package_DIP:DIP-14_W7.62mm_Socket_LongPads -> Custom:STD_DDW_DIP14
- U2, U3: footprint Package_DIP:DIP-20_W7.62mm_Socket_LongPads -> Custom:STD_DDW_DIP20
- U23: value 74LS138 -> 74LS688; footprint Package_DIP:DIP-16_W7.62mm_Socket_LongPads -> Custom:STD_DDW_DIP20
- U25: renamed from U24; footprint Package_DIP:DIP-20_W7.62mm_Socket_LongPads -> Custom:STD_DDW_DIP20
- U26: renamed from U25; footprint Package_DIP:DIP-20_W7.62mm_Socket_LongPads -> Custom:STD_DDW_DIP20
- U27: renamed from U26; footprint Package_DIP:DIP-20_W7.62mm_Socket_LongPads -> Custom:STD_DDW_DIP20
- U28: renamed from U27; footprint Package_DIP:DIP-20_W7.62mm_Socket_LongPads -> Custom:STD_DDW_DIP20
- U29: renamed from U28; footprint Package_TO_SOT_THT:TO-92L_HandSolder -> Custom:STD_DDW_TO92
- U30: renamed from U29; footprint Package_DIP:DIP-16_W7.62mm_Socket_LongPads -> Custom:STD_DDW_DIP16
- U31: renamed from U30; footprint Package_DIP:DIP-20_W7.62mm_Socket_LongPads -> Custom:STD_DDW_DIP20
- U32: renamed from U31; footprint Package_DIP:DIP-20_W7.62mm_Socket_LongPads -> Custom:STD_DDW_DIP20
- U33: renamed from U32; footprint Package_DIP:DIP-40_W15.24mm_Socket_LongPads -> Custom:STD_DDW_DIP40
- U34: renamed from U33; footprint Package_DIP:DIP-20_W7.62mm_Socket_LongPads -> Custom:STD_DDW_DIP20
- U35: renamed from U34; footprint Package_DIP:DIP-16_W7.62mm_Socket_LongPads -> Custom:STD_DDW_DIP16
- U36: renamed from U35; footprint Package_DIP:DIP-20_W7.62mm_Socket_LongPads -> Custom:STD_DDW_DIP20
- U37: renamed from U36; footprint Package_DIP:DIP-16_W7.62mm_Socket_LongPads -> Custom:STD_DDW_DIP16
- U38: renamed from U37; footprint Package_DIP:DIP-20_W7.62mm_Socket_LongPads -> Custom:STD_DDW_DIP20
- U39: renamed from U38; footprint Package_DIP:DIP-20_W7.62mm_Socket_LongPads -> Custom:STD_DDW_DIP20
- U40: renamed from U39; footprint Package_DIP:DIP-28_W7.62mm_Socket_LongPads -> Custom:STD_DDW_DIP28_SKINNY
- U41: renamed from U40; footprint Package_DIP:DIP-20_W7.62mm_Socket_LongPads -> Custom:STD_DDW_DIP20
- U42: renamed from U41; footprint Package_DIP:DIP-16_W7.62mm_Socket_LongPads -> Custom:STD_DDW_DIP16
- U43: renamed from U42; footprint Package_DIP:DIP-16_W7.62mm_Socket_LongPads -> Custom:STD_DDW_DIP16
- U44: renamed from U43; footprint Package_DIP:DIP-16_W7.62mm_Socket_LongPads -> Custom:STD_DDW_DIP16
- U45: renamed from U44; footprint Package_DIP:DIP-20_W7.62mm_Socket_LongPads -> Custom:STD_DDW_DIP20
- U46: renamed from U45; footprint Package_DIP:DIP-20_W7.62mm_Socket_LongPads -> Custom:STD_DDW_DIP20
- U47: renamed from U46; footprint Package_DIP:DIP-18_W7.62mm_Socket_LongPads -> Custom:STD_DDW_DIP18
- U48: renamed from U47; footprint Package_DIP:DIP-28_W15.24mm_Socket_LongPads -> Custom:STD_DDW_DIP28
- U49: renamed from U48; footprint Package_DIP:DIP-16_W7.62mm_Socket_LongPads -> Custom:STD_DDW_DIP16
- U50: renamed from U49; footprint Package_DIP:DIP-16_W7.62mm_Socket_LongPads -> Custom:STD_DDW_DIP16
- U51: renamed from U50; footprint Package_DIP:DIP-16_W7.62mm_Socket_LongPads -> Custom:STD_DDW_DIP16
- U52: renamed from U51; footprint Package_DIP:DIP-16_W7.62mm_Socket_LongPads -> Custom:STD_DDW_DIP16
- U53: renamed from U52; footprint Package_DIP:DIP-16_W7.62mm_Socket_LongPads -> Custom:STD_DDW_DIP16
- U56: renamed from U55; footprint Package_DIP:DIP-20_W7.62mm_Socket_LongPads -> Custom:STD_DDW_DIP20
- U57: renamed from U56; footprint Package_DIP:DIP-40_W15.24mm_Socket_LongPads -> Custom:STD_DDW_DIP40
- U58: renamed from U57; footprint Package_DIP:DIP-40_W15.24mm_Socket_LongPads -> Custom:STD_DDW_DIP40
- U8, U9: footprint Package_DIP:DIP-32_W15.24mm_Socket_LongPads -> Custom:STD_DDW_DIP32
- X1: footprint Crystal:Crystal_DS10_D1.0mm_L4.3mm_Horizontal -> Custom:DDW_STD_RTCCRYSTAL
- moved C48 628.5 mm to (85.4, 162.6), turned to 0 degrees
- moved C46 597.7 mm to (105.4, 162.0), turned to 0 degrees
- moved C31 567.4 mm to (96.9, 256.2), turned to 0 degrees
- moved C29 566.9 mm to (125.8, 161.0), turned to 0 degrees
- moved U30 558.2 mm to (146.7, 240.3), turned to 0 degrees
- moved C9 550.0 mm to (84.9, 188.1), turned to 0 degrees
- moved U8 549.6 mm to (83.9, 261.9), turned to 0 degrees
- moved C42 544.4 mm to (102.0, 188.2), turned to 0 degrees
- moved P14 544.3 mm to (146.8, 273.4), turned to 0 degrees
- moved C52 538.7 mm to (119.3, 187.9), turned to 0 degrees
- moved C43 537.4 mm to (144.5, 161.1), turned to 0 degrees
- moved C58 534.7 mm to (146.5, 257.9), turned to 0 degrees
- moved C11 532.8 mm to (137.1, 186.8), turned to 0 degrees
- moved U9 528.0 mm to (125.9, 261.9), turned to 0 degrees
- moved C49 527.5 mm to (153.9, 187.0), turned to 0 degrees
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- renumbered J8 to J16, J9 to J17, J2 to J8, P7 to P11, U53 to U54, U54 to U55
Connections:
- net isa_iq_2 renamed isa_iq_3
- U1 pad 12: Net-(U23-E2) -> Net-(U1-Pad12)
- U1 pad 3: /MMU four//MMU-MAP-RW -> /IOSEL-0EFD0
- U10 pad 10: unconnected-(U10-Pad10) -> /IOSEL-0EFD0
- U10 pad 11: unconnected-(U10-Pad11) -> /MMU four//MMU-MAP-RD
- U10 pad 12: unconnected-(U10-Pad12) -> /IOSEL-0EFD0
- U10 pad 13: unconnected-(U10-Pad13) -> CPU_/RD
- U10 pad 8: unconnected-(U10-Pad8) -> /MMU four//MMU-MAP-WR
- U10 pad 9: unconnected-(U10-Pad9) -> CPU_/WR
- U11 pad 1: /IOSEL-0EBxx -> /IOSEL-0EFC0
- U11 pad 12: /IOSEL-0EBxx -> /IOSEL-0EFC0
- U11 pad 9: /IOSEL-0EBxx -> /IOSEL-0EFC0
- U15 pad 11: /MMU four//MMU-MAP-RW -> unconnected-(U15-Pad11)
- U15 pad 12: /MMU four//MMU-MAP-RD -> unconnected-(U15-Pad12)
- U15 pad 13: /MMU four//MMU-MAP-WR -> unconnected-(U15-Pad13)
- U21 pad 5: Net-(U23-E2) -> Net-(U1-Pad12)
- U23 pad 1: mA8 -> /VMA
- U23 pad 10: /IOSEL-0EDxx -> GND
- U23 pad 11: /IOSEL-0ECxx -> mA9
- U23 pad 12: /IOSEL-0EBxx -> VCC
- U23 pad 13: /IOSEL-0EAxx -> mA8
- U23 pad 14: /IOSEL-0E9xx -> VCC
- U23 pad 15: /IOSEL-0E8xx -> mA7
- U23 pad 16: GND -> VCC
- U23 pad 2: mA9 -> SHADOW-IO
- U23 pad 3: mA10 -> VCC
- U23 pad 4: /VMA -> VCC
- U23 pad 5: Net-(U23-E2) -> VCC
- U23 pad 6: SHADOW-IO -> mA11
- U23 pad 7: /IOSEL-0EFxx -> VCC
- U23 pad 8: VCC -> mA10
- U23 pad 9: /IOSEL-0EExx -> VCC
- U38 pad 1: /MMU four//MMU-MAP-RW -> /IOSEL-0EFD0
- U41 pad 19: /MMU four//MMU-MAP-RW -> /IOSEL-0EFD0
- U42 pad 1: mA4 -> mA0
- U42 pad 12: /MMU four//MMU-ENB-WR -> unconnected-(U42-O3-Pad12)
- U42 pad 13: /MMU four//MMU-MAP-WR -> /MMU four//MMU-ENB-WR
- U42 pad 2: mA5 -> mA1
- U42 pad 4: /IOSEL-0EAxx -> /IOSEL-0EFE0
- U42 pad 9: /MMU four//MMU-MAP-RD -> unconnected-(U42-O6-Pad9)
- U47 pad 2: /IOSEL-0EExx -> /IOSEL-0EF90
- U48 pad 3: /IOSEL-0EFxx -> /IOSEL-0EF80
- U57 pad 23: /IOSEL-0ECxx -> /IOSEL-0EFA0
- U58 pad 23: /IOSEL-0EDxx -> /IOSEL-0EFB0
Other:
- board size 233.7 x 160 mm -> 244 x 244 mm
- board text added: "6809PC ATX rev. 1.00-000 1/21/2025 D. Werner https://github.com/danwerner21/6809PC Licensed for hobbyist use only. All other rights reserved."
- board text added: "8Mhz 1-2 4Mhz 3-4 2Mhz 5-6 1Mhz 7-8"
- board text added: "VERIFY ISA PINOUTS VERIFY CONNECTOR PINOUTS VERIFY ATXPOWER PINOUTS"
- board text removed: "6809PC ATX/VME rev. 2.00-012 Copyright (C) 2014 Andrew Lynch & John Coffman. Licensed for hobbyist use only. All other rights reserved."
- board text removed: "ATX Connector Area"
- board text removed: "ATX hole pattern displaced 0.030""
- board text removed: "Centers of holes made to overlap"
- board text removed: "ECB 3U connector area"
- board text removed: "Eurocard 6U drilled to fit an ATX chassis"
- board text removed: "UNIVERSAL"
