File: ESP_IO.kicad_sch (KiCad schematic)
At the start: 45 parts, among them J10 AUDIO OUT, J11 TTL SERIAL 0, J12 TTL SER 0 PWR, J13 TTL SERIAL 1, J14 TTL SER 1 PWR, J5 KEYBOARD AND MOUSE, J6 VGA, J7 VGA, J8 Keyboard, J9 Mouse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

Commit message: PCB in progress
Parts:
- C67: footprint Capacitor_THT:C_Disc_D5.0mm_W2.5mm_P5.00mm -> Custom:STD_DDW_CAP
- C68: footprint Capacitor_THT:CP_Radial_D5.0mm_P2.50mm -> Custom:STD_DDW_PCAP
- D5, D6: footprint Diode_THT:D_DO-41_SOD81_P10.16mm_Horizontal -> Custom:STD_DDW_DIODE
- J13: renamed from J5; footprint Connector_PinHeader_2.54mm:PinHeader_2x05_P2.54mm_Horizontal -> Custom:STD_DDW_PINHEAD_V_2x05
- J14: renamed from J6; footprint Connector_Dsub:DSUB-15-HD_Female_Horizontal_P2.29x1.98mm_EdgePinOffset3.03mm_Housed_MountingHolesOffset4.94mm -> Custom:STD_DDW_VGA
- J15: renamed from J7; footprint Connector_PinHeader_2.54mm:PinHeader_1x07_P2.54mm_Horizontal -> Custom:STD_DDW_PINHEAD_V_1x07
- J18: renamed from J10; footprint Connector_PinHeader_2.54mm:PinHeader_1x02_P2.54mm_Horizontal -> Custom:STD_DDW_PINHEAD_V_1x02
- J19: renamed from J11; footprint Connector_PinHeader_2.54mm:PinHeader_1x06_P2.54mm_Horizontal -> Custom:STD_DDW_PINHEAD_V_1x06
- J20: renamed from J12; footprint Connector_PinHeader_2.54mm:PinHeader_1x02_P2.54mm_Vertical -> Custom:STD_DDW_PINHEAD_V_1x02
- J21: renamed from J13; footprint Connector_PinHeader_2.54mm:PinHeader_1x06_P2.54mm_Horizontal -> Custom:STD_DDW_PINHEAD_V_1x06
- J22: renamed from J14; footprint Connector_PinHeader_2.54mm:PinHeader_1x02_P2.54mm_Vertical -> Custom:STD_DDW_PINHEAD_V_1x02
- R10, R11, R12, R13, R14, R15, R16, R17, R18, R19, R20, R21, R22, R23, R8, R9: footprint Resistor_THT:R_Axial_DIN0207_L6.3mm_D2.5mm_P7.62mm_Horizontal -> Custom:STD_DDW_RESISTOR
- RN1: footprint Resistor_THT:R_Array_SIP9 -> Custom:STD_DDW_SIP9
- U10, U11, U12, U13, U14, U16, U20: footprint Package_DIP:DIP-14_W7.62mm_Socket_LongPads -> Custom:STD_DDW_DIP14
- U50: renamed from U49; footprint Package_DIP:DIP-16_W7.62mm_Socket_LongPads -> Custom:STD_DDW_DIP16
- U51: renamed from U50; footprint Package_DIP:DIP-16_W7.62mm_Socket_LongPads -> Custom:STD_DDW_DIP16
- U52: renamed from U51; footprint Package_DIP:DIP-16_W7.62mm_Socket_LongPads -> Custom:STD_DDW_DIP16
- U53: renamed from U52; footprint Package_DIP:DIP-16_W7.62mm_Socket_LongPads -> Custom:STD_DDW_DIP16
- U56: renamed from U55; footprint Package_DIP:DIP-20_W7.62mm_Socket_LongPads -> Custom:STD_DDW_DIP20
- renumbered J8 to J16, J9 to J17, U53 to U54, U54 to U55
Connections:
- net /IOSEL-0EBxx renamed /IOSEL-0EFC0
