File: VIAS.kicad_sch (KiCad schematic)
At the start: 7 parts, among them K3 CONN_3, P16 CONN_8X2, P17 PARALLEL

Commit message: Schematic in progress
Parts:
- added JP4: JUMPER, Connector_PinHeader_2.54mm:PinHeader_1x02_P2.54mm_Vertical, symbol Jumper:Jumper_2_Open
- added R24: 22K, Resistor_THT:R_Axial_DIN0207_L6.3mm_D2.5mm_P7.62mm_Horizontal, symbol Device:R
- JP5: footprint PIN_ARRAY_2X1 -> Connector_PinHeader_2.54mm:PinHeader_1x02_P2.54mm_Vertical
- K3: footprint PIN_ARRAY_3X1 -> Connector_PinHeader_2.54mm:PinHeader_1x03_P2.54mm_Vertical
- P15: renamed from P16; footprint PIN_ARRAY_8x2 -> Connector_PinHeader_2.54mm:PinHeader_2x08_P2.54mm_Vertical
- P16: renamed from P17; footprint PIN_ARRAY_13x2 -> Connector_PinHeader_2.54mm:PinHeader_2x13_P2.54mm_Vertical
- R25: renamed from R11; footprint R3 -> Resistor_THT:R_Axial_DIN0207_L6.3mm_D2.5mm_P7.62mm_Horizontal
- U? (x2): footprint Package_DIP:DIP-40_W15.24mm -> Package_DIP:DIP-40_W15.24mm_Socket_LongPads
Connections:
- net CA1: now also P15.3 (Pin_3); no longer P15.1 (Pin_1)
- net CA2: now also P15.5 (Pin_5); no longer P15.3 (Pin_3)
- net CB1: now also P15.7 (Pin_7); no longer P15.5 (Pin_5)
- net CB2: now also P15.9 (Pin_9); no longer P15.7 (Pin_7)
- net CC1: now also P15.11 (Pin_11); no longer P15.9 (Pin_9)
- net CC2: now also P15.13 (Pin_13); no longer P15.11 (Pin_11)
- net CD1: now also JP4.2 (B), R24.2; no longer P15.13 (Pin_13)
- net GND: now also JP4.1 (A)
- net PD0: now also P15.2 (Pin_2)
- net VCC: now also P15.1 (Pin_1), R24.1; no longer P15.2 (Pin_2)
Other:
- company: N8VEM Users Group -> (none)
- title: 6809 and 6502 ATX and 6U -> 6809PC

Commit message: PCB in progress
Parts:
- JP4: value JUMPER -> OPT1; footprint Connector_PinHeader_2.54mm:PinHeader_1x02_P2.54mm_Vertical -> Custom:STD_DDW_PINHEAD_V_1x02
- JP5: value JUMPER -> OPT2; footprint Connector_PinHeader_2.54mm:PinHeader_1x02_P2.54mm_Vertical -> Custom:STD_DDW_PINHEAD_V_1x02
- K3: value CONN_3 -> P Port Power; footprint Connector_PinHeader_2.54mm:PinHeader_1x03_P2.54mm_Vertical -> Custom:STD_DDW_PINHEAD_V_1x03
- P19: renamed from P15; value CONN_8X2 -> VIA OUTPUT; footprint Connector_PinHeader_2.54mm:PinHeader_2x08_P2.54mm_Vertical -> Custom:STD_DDW_PINHEAD_V_2x08
- P20: renamed from P16; footprint Connector_PinHeader_2.54mm:PinHeader_2x13_P2.54mm_Vertical -> Custom:STD_DDW_PINHEAD_V_2x13
- R24, R25: footprint Resistor_THT:R_Axial_DIN0207_L6.3mm_D2.5mm_P7.62mm_Horizontal -> Custom:STD_DDW_RESISTOR
- U? (x2): footprint Package_DIP:DIP-40_W15.24mm_Socket_LongPads -> Custom:STD_DDW_DIP40
Connections:
- net /IOSEL-0ECxx renamed /IOSEL-0EFA0
- net /IOSEL-0EDxx renamed /IOSEL-0EFB0
