File: 6809PC-6U.kicad_sch (KiCad schematic)
At the start: 0 parts

Commit message: Schematic in progress
Other:
- sheet ECB bus renamed ISA bus
- added sheet ESP_IO (ESP_IO.kicad_sch)
- note removed: "Need Video (ESP32)"
- note removed: "New RTC"
- note removed: "STD TTL Serial Connector"
- note removed: "change to ISA"
- company: N8VEM Users Group -> (none)
- title: 6809 and 6502 ATX and 6U -> 6809PC
Changed lines of the file:
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@@
 	(paper "A")
 	(title_block
-		(title "6809 and 6502 ATX and 6U")
-		(date "19 feb 2014")
-		(rev "012")
-		(company "N8VEM Users Group")
-		(comment 1 "Licensed for hobbyist use only.  All other rights reserved.")
-		(comment 2 "Copyright (c) 2013-2014  Andrew Lynch and John Coffman")
-	)
-	(text "change to ISA"
+		(title "6809PC")
+		(date "2025-01-21")
+		(rev "001")
+		(comment 1 "https://github.com/danwerner21/6809PC")
+		(comment 2 "Based on work by Andrew Lynch and John Coffman")
+	)
+	(text "Better IO Decoding"
 		(exclude_from_sim no)
-		(at 35.814 59.69 0)
+		(at 34.036 121.412 0)
 		(effects
 			(font
@@
 		)
 	)
-	(text "Need Video (ESP32)"
-		(exclude_from_sim no)
-		(at 36.068 56.134 0)
-		(effects
-			(font
-				(size 2.032 2.032)
-				(thickness 0.4064)
-				(bold yes)
-			)
-			(justify left bottom)
-		)
-	)
-	(text "New RTC"
-		(exclude_from_sim no)
-		(at 36.322 67.818 0)
-		(effects
-			(font
-				(size 2.032 2.032)
-				(thickness 0.4064)
-				(bold yes)
-			)
-			(justify left bottom)
-		)
-	)
-	(text "STD TTL Serial Connector"
-		(exclude_from_sim no)
-		(at 36.068 71.12 0)
-		(effects
-			(font
-				(size 2.032 2.032)
-				(thickness 0.4064)
-				(bold yes)
-			)
-			(justify left bottom)
-		)
-	)
-	(text "Better IO Decoding"
-		(exclude_from_sim no)
-		(at 36.068 63.754 0)
-		(effects
-			(font
-				(size 2.032 2.032)
-				(thickness 0.4064)
-				(bold yes)
-			)
-			(justify left bottom)
-		)
-	)
 	(sheet
 		(at 30.48 29.21)
@@
 			(color 0 0 0 0.0000)
 		)
-		(property "Sheetname" "ECB bus"
+		(property "Sheetname" "ISA bus"
 			(at 30.48 28.3714 0)
 			(effects
@@
 	)
 	(sheet
-		(at 114.3 60.96)
+		(at 113.03 29.21)
 		(size 25.4 15.24)
 		(fields_autoplaced yes)
@@
 		)
 		(property "Sheetname" "MMU four"
-			(at 114.3 60.1214 0)
+			(at 113.03 28.3714 0)
 			(effects
 				(font
@@
 		)
 		(property "Sheetfile" "MMU-4.kicad_sch"
-			(at 114.3 76.8862 0)
+			(at 113.03 45.1362 0)
 			(effects
 				(font
@@
 	)
 	(sheet
-		(at 30.48 156.21)
+		(at 30.48 58.42)
 		(size 25.4 15.24)
 		(fields_autoplaced yes)
@@
 		)
 		(property "Sheetname" "Power"
-			(at 30.48 155.3714 0)
+			(at 30.48 57.5814 0)
 			(effects
 				(font
@@
 		)
 		(property "Sheetfile" "Power.kicad_sch"
-			(at 30.48 172.1362 0)
+			(at 30.48 74.3462 0)
 			(effects
 				(font
@@
 	)
 	(sheet
-		(at 72.39 127)
+		(at 113.03 59.69)
 		(size 25.4 15.24)
 		(fields_autoplaced yes)
@@
 		)
 		(property "Sheetname" "Spare"
-			(at 72.39 126.1614 0)
+			(at 113.03 58.8514 0)
 			(effects
 				(font
@@
 		)
 		(property "Sheetfile" "Spare.kicad_sch"
-			(at 72.39 142.9262 0)
+			(at 113.03 75.6162 0)
 			(effects
 				(font
@@
 	)
 	(sheet
-		(at 72.39 156.21)
+		(at 114.3 90.17)
 		(size 25.4 15.24)
 		(fields_autoplaced yes)
@@
 		)
 		(property "Sheetname" "Reset"
-			(at 72.39 155.3714 0)
+			(at 114.3 89.3314 0)
 			(effects
 				(font
@@
 		)
 		(property "Sheetfile" "Reset.kicad_sch"
-			(at 72.39 172.1362 0)
+			(at 114.3 106.0962 0)
 			(effects
 				(font
@@
 				)
 			)
+		)
+	)
+	(sheet
+		(at 198.12 29.21)
+		(size 24.13 16.51)
+		(fields_autoplaced yes)
+		(stroke
+			(width 0.1524)
+			(type solid)
+		)
+		(fill
+			(color 0 0 0 0.0000)
+		)
+		(property "Sheetname" "ESP_IO"
+			(at 198.12 28.4984 0)
+			(effects
+				(font
+					(size 1.27 1.27)
+				)
+				(justify left bottom)
+			)
+		)
+		(property "Sheetfile" "ESP_IO.kicad_sch"
+			(at 198.12 46.3046 0)
+			(effects
+				(font
+					(size 1.27 1.27)
+				)
+				(justify left top)
+			)
+		)
+		(instances
+			(project "6809PC-6U"
+				(path "/d94f9d60-5ece-4752-b49c-b0d1c95f35bc"
+					(page "14")
+				)
+			)

Commit message: PCB in progress
Other:
- note removed: "Better IO Decoding"
Changed lines of the file:
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@@
 		(comment 2 "Based on work by Andrew Lynch and John Coffman")
-	)
-	(text "Better IO Decoding"
-		(exclude_from_sim no)
-		(at 34.036 121.412 0)
-		(effects
-			(font
-				(size 2.032 2.032)
-				(thickness 0.4064)
-				(bold yes)
-			)
-			(justify left bottom)
-		)
 	)
 	(sheet

Commit message: 6809PC work
Other:
- removed sheet ESP_IO
- removed sheet VIAS
Changed lines of the file:
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@@
 	(title_block
 		(title "6809PC")
-		(date "2025-01-21")
-		(rev "001")
+		(date "2025-05-17")
+		(rev "002")
 		(comment 1 "https://github.com/danwerner21/6809PC")
 		(comment 2 "Based on work by Andrew Lynch and John Coffman")
@@
 	)
 	(sheet
-		(at 156.21 91.44)
-		(size 25.4 15.24)
-		(fields_autoplaced yes)
-		(stroke
-			(width 0)
-			(type solid)
-		)
-		(fill
-			(color 0 0 0 0.0000)
-		)
-		(property "Sheetname" "VIAS"
-			(at 156.21 90.6014 0)
-			(effects
-				(font
-					(size 1.524 1.524)
-				)
-				(justify left bottom)
-			)
-		)
-		(property "Sheetfile" "VIAS.kicad_sch"
-			(at 156.21 107.3662 0)
-			(effects
-				(font
-					(size 1.524 1.524)
-				)
-				(justify left top)
-			)
-		)
-		(instances
-			(project "6809PC-6U"
-				(path "/d94f9d60-5ece-4752-b49c-b0d1c95f35bc"
-					(page "15")
-				)
-			)
-		)
-	)
-	(sheet
 		(at 156.21 29.21)
 		(size 25.4 15.24)
@@
 				)
 			)
-		)
-	)
-	(sheet
-		(at 198.12 29.21)
-		(size 24.13 16.51)
-		(fields_autoplaced yes)
-		(stroke
-			(width 0.1524)
-			(type solid)
-		)
-		(fill
-			(color 0 0 0 0.0000)
-		)
-		(property "Sheetname" "ESP_IO"
-			(at 198.12 28.4984 0)
-			(effects
-				(font
-					(size 1.27 1.27)
-				)
-				(justify left bottom)
-			)
-		)
-		(property "Sheetfile" "ESP_IO.kicad_sch"
-			(at 198.12 46.3046 0)
-			(effects
-				(font
-					(size 1.27 1.27)
-				)
-				(justify left top)
-			)
-		)
-		(instances
-			(project "6809PC-6U"
-				(path "/d94f9d60-5ece-4752-b49c-b0d1c95f35bc"
-					(page "14")
-				)
-			)
