File: ACIA.kicad_sch (KiCad schematic)
At the start: 16 parts, among them P13 1.8432 MHz CLK, P14 SERIAL, P15 CONN_5X2, U44 MAX232

Commit message: Schematic in progress
Parts:
- removed P15: CONN_5X2, PIN_ARRAY_5x2, symbol Connector_Generic:Conn_02x05_Odd_Even
- added J3: TTL SERIAL CONSOLE, Connector_PinHeader_2.54mm:PinHeader_1x06_P2.54mm_Horizontal, symbol Connector_Generic:Conn_01x06
- added J4: TTL CONSOLE PWR, Connector_PinHeader_2.54mm:PinHeader_1x02_P2.54mm_Vertical, symbol Connector_Generic:Conn_01x02
- C61: renamed from C58; footprint C1V5 -> Capacitor_THT:CP_Radial_D5.0mm_P2.50mm
- C62: renamed from C59; footprint C2 -> Capacitor_THT:C_Disc_D5.0mm_W2.5mm_P5.00mm
- C63: renamed from C60; footprint C1V5 -> Capacitor_THT:CP_Radial_D5.0mm_P2.50mm
- C64: renamed from C61; footprint C1V5 -> Capacitor_THT:CP_Radial_D5.0mm_P2.50mm
- C65: renamed from C62; footprint C1V5 -> Capacitor_THT:CP_Radial_D5.0mm_P2.50mm
- C66: renamed from C63; footprint C1V5 -> Capacitor_THT:CP_Radial_D5.0mm_P2.50mm
- JP3: renamed from JP4; footprint PIN_ARRAY_2X1 -> Connector_PinHeader_2.54mm:PinHeader_1x02_P2.54mm_Vertical
- P13: footprint DIP-14__300 -> Package_DIP:DIP-14_W7.62mm_Socket_LongPads
- P14: footprint PIN_ARRAY_5x2 -> Connector_PinHeader_2.54mm:PinHeader_2x05_P2.54mm_Vertical
- R4: renamed from R7; footprint R3 -> Resistor_THT:R_Axial_DIN0207_L6.3mm_D2.5mm_P7.62mm_Horizontal
- R5: renamed from R8; footprint R3 -> Resistor_THT:R_Axial_DIN0207_L6.3mm_D2.5mm_P7.62mm_Horizontal
- R6: renamed from R9; footprint R3 -> Resistor_THT:R_Axial_DIN0207_L6.3mm_D2.5mm_P7.62mm_Horizontal
- R7: renamed from R10; footprint R3 -> Resistor_THT:R_Axial_DIN0207_L6.3mm_D2.5mm_P7.62mm_Horizontal
- U48: renamed from U44; footprint DIP-16__300 -> Package_DIP:DIP-16_W7.62mm_Socket_LongPads
- U?: footprint Package_DIP:DIP-28_W15.24mm -> Package_DIP:DIP-28_W15.24mm_Socket_LongPads
Connections:
- net GND: now also J3.1 (Pin_1)
- net RXD_TTL: now also J3.4 (Pin_4)
- net TXD_TTL: now also J3.5 (Pin_5)
- net VCC: now also J4.1 (Pin_1)
- net RXCLK: no longer names the net of U?.5 (RxC)
- new net: J3.3 (Pin_3), J4.2 (Pin_2)
- no-connect marks 11 -> 14
Other:
- company: N8VEM Users Group -> (none)
- title: 6809 and 6502 ATX and 6U -> 6809PC

Commit message: PCB in progress
Parts:
- C61, C63, C64, C65, C66: footprint Capacitor_THT:CP_Radial_D5.0mm_P2.50mm -> Custom:STD_DDW_PCAP
- C62: footprint Capacitor_THT:C_Disc_D5.0mm_W2.5mm_P5.00mm -> Custom:STD_DDW_CAP
- J11: renamed from J3; footprint Connector_PinHeader_2.54mm:PinHeader_1x06_P2.54mm_Horizontal -> Custom:STD_DDW_PINHEAD_V_1x06
- J12: renamed from J4; footprint Connector_PinHeader_2.54mm:PinHeader_1x02_P2.54mm_Vertical -> Custom:STD_DDW_PINHEAD_V_1x02
- JP3: footprint Connector_PinHeader_2.54mm:PinHeader_1x02_P2.54mm_Vertical -> Custom:STD_DDW_PINHEAD_V_1x02
- P17: renamed from P13; footprint Package_DIP:DIP-14_W7.62mm_Socket_LongPads -> Custom:STD_DDW_DIP14
- P18: renamed from P14; footprint Connector_PinHeader_2.54mm:PinHeader_2x05_P2.54mm_Vertical -> Custom:STD_DDW_PINHEAD_V_2x05
- R4, R5, R6, R7: footprint Resistor_THT:R_Axial_DIN0207_L6.3mm_D2.5mm_P7.62mm_Horizontal -> Custom:STD_DDW_RESISTOR
- U49: renamed from U48; footprint Package_DIP:DIP-16_W7.62mm_Socket_LongPads -> Custom:STD_DDW_DIP16
- U?: footprint Package_DIP:DIP-28_W15.24mm_Socket_LongPads -> Custom:STD_DDW_DIP28
Connections:
- net /IOSEL-0EFxx renamed /IOSEL-0EF80

Commit message: 6809PC work
Connections:
- net CTS_TTL: now also J11.6 (Pin_6)
- net RTS_TTL: now also J11.2 (Pin_2)
- no-connect marks 14 -> 12
Changed lines of the file:
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@@
 	(title_block
 		(title "6809PC")
-		(date "2025-01-21")
-		(rev "001")
+		(date "2025-05-17")
+		(rev "002")
 		(comment 1 "https://github.com/danwerner21/6809PC")
 		(comment 2 "Based on work by Andrew Lynch and John Coffman")
@@
 	)
 	(no_connect
-		(at 212.09 110.49)
-	)
-	(no_connect
 		(at 213.36 142.24)
 	)
@@
 	)
 	(no_connect
-		(at 212.09 100.33)
-	)
-	(no_connect
 		(at 104.14 36.83)
 	)
@@
 	(wire
 		(pts
+			(xy 212.09 100.33) (xy 217.17 100.33)
+		)
+		(stroke
+			(width 0)
+			(type default)
+		)
+	)
+	(wire
+		(pts
 			(xy 229.87 63.5) (xy 222.25 63.5)
 		)
@@
 	(wire
 		(pts
+			(xy 212.09 110.49) (xy 226.06 110.49)
+		)
+		(stroke
+			(width 0)
+			(type default)
+		)
+	)
+	(wire
+		(pts
 			(xy 60.96 146.05) (xy 60.96 151.13)
 		)
@@
 	(wire
 		(pts
-			(xy 212.09 97.79) (xy 215.9 97.79)
+			(xy 212.09 97.79) (xy 222.25 97.79)
 		)
 		(stroke
@@
 		)
 	)
+	(label "RTS_TTL"
+		(at 212.09 100.33 0)
+		(fields_autoplaced yes)
+		(effects
+			(font
+				(size 1.524 1.524)
+			)
+			(justify left bottom)
+		)
+	)
 	(label "CTS"
 		(at 229.87 68.58 180)
@@
 			(font
 				(size 1.524 1.524)
+			)
+			(justify left bottom)
+		)
+	)
+	(label "CTS_TTL"
+		(at 218.44 110.49 0)
+		(fields_autoplaced yes)
+		(effects
+			(font
+				(size 1.27 1.27)
 			)
 			(justify left bottom)
@@
 	(symbol
 		(lib_id "power:GND")
-		(at 215.9 97.79 0)
+		(at 222.25 97.79 0)
 		(unit 1)
 		(exclude_from_sim no)
@@
 		(dnp no)
 		(property "Reference" "#PWR0161"
-			(at 215.9 97.79 0)
+			(at 222.25 97.79 0)
 			(effects
 				(font
@@
 		)
 		(property "Value" "GND"
-			(at 215.9 99.568 0)
+			(at 222.25 99.568 0)
 			(effects
 				(font
@@
 		)
 		(property "Footprint" ""
-			(at 215.9 97.79 0)
+			(at 222.25 97.79 0)
 			(effects
 				(font
@@
 		)
 		(property "Datasheet" ""
-			(at 215.9 97.79 0)
+			(at 222.25 97.79 0)
 			(effects
 				(font
@@
 		)
 		(property "Description" "Power symbol creates a global label with name \"GND\" , ground"
-			(at 215.9 97.79 0)
-			(effects
-				(font
+			(at 222.25 97.79 0)
+			(effects
+				(font
