File: IO.kicad_sch (KiCad schematic)
At the start: 8 parts, among them U12 74LS00, U15 74LS245, U16 74LS245, U17 74LS245, U18 74LS245, U4 74LS86, U6 74LS00

Commit message: Schematic in progress
Parts:
- added C56: 0.1 uF, Capacitor_THT:C_Disc_D5.0mm_W2.5mm_P5.00mm, symbol Device:C
- added P9: 14.31818 MHz CLK, Package_DIP:DIP-14_W7.62mm_Socket_LongPads, symbol Custom:CLK
- added U16, U7: 74LS32, Package_DIP:DIP-14_W7.62mm_Socket_LongPads, symbol 74xx:74LS32
- added U17: 74LS14, Package_DIP:DIP-14_W7.62mm_Socket_LongPads, symbol 74xx:74LS14
- added U18: 74LS06, Package_DIP:DIP-14_W7.62mm_Socket_LongPads, symbol 74xx:74LS06
- U21: renamed from U12; footprint DIP-14__300 -> Package_DIP:DIP-14_W7.62mm_Socket_LongPads
- U24: renamed from U15; footprint DIP-20__300 -> Package_DIP:DIP-20_W7.62mm_Socket_LongPads
- U25: renamed from U16; footprint DIP-20__300 -> Package_DIP:DIP-20_W7.62mm_Socket_LongPads
- U26: renamed from U17; footprint DIP-20__300 -> Package_DIP:DIP-20_W7.62mm_Socket_LongPads
- U27: renamed from U18; footprint DIP-20__300 -> Package_DIP:DIP-20_W7.62mm_Socket_LongPads
- U4, U6: footprint DIP-14__300 -> Package_DIP:DIP-14_W7.62mm_Socket_LongPads
Connections:
- net B_/INT: now also U18.12
- net B_/MREQ: now also U16.1, U16.9
- net B_/RD: now also U16.10, U16.5
- net B_/WR: now also U16.2, U7.13
- net GND: now also C56.2, P9.4, P9.5, P9.6, P9.7
- net VCC: now also C56.1, P9.14
- net /PG renamed PULLUP3
- net B_/M1 renamed PULLUP4
- net B_/WAIT renamed PULLUP2
- net SD_SEL renamed PULLUP1
- new net BUSALE: U17.2
- new net BUSCLK: P9.10, P9.11, P9.8, P9.9
- new net B_/IORQ: U16.4, U7.12
- new net B_INT: U18.13
- new net CPU_Q: U17.1
- new net IOR: U16.8
- new net IOW: U16.6
- new net SMEMR: U16.3
- new net SMEMW: U7.11
- no-connect marks 3 -> 8
Other:
- note added: "Bus Address Latch Enable. The address bus is latched on the rising edge of this signal."
- company: N8VEM Users Group -> (none)
- title: 6809 and 6502 ATX and 6U -> 6809PC

Commit message: PCB in progress
Parts:
- C56: footprint Capacitor_THT:C_Disc_D5.0mm_W2.5mm_P5.00mm -> Custom:STD_DDW_CAP
- P13: renamed from P9; footprint Package_DIP:DIP-14_W7.62mm_Socket_LongPads -> Custom:STD_DDW_DIP14
- RR1: footprint Resistor_THT:R_Array_SIP10 -> Custom:STD_DDW_SIP10
- U16, U17, U18, U21, U4, U6, U7: footprint Package_DIP:DIP-14_W7.62mm_Socket_LongPads -> Custom:STD_DDW_DIP14
- U25: renamed from U24; footprint Package_DIP:DIP-20_W7.62mm_Socket_LongPads -> Custom:STD_DDW_DIP20
- U26: renamed from U25; footprint Package_DIP:DIP-20_W7.62mm_Socket_LongPads -> Custom:STD_DDW_DIP20
- U27: renamed from U26; footprint Package_DIP:DIP-20_W7.62mm_Socket_LongPads -> Custom:STD_DDW_DIP20
- U28: renamed from U27; footprint Package_DIP:DIP-20_W7.62mm_Socket_LongPads -> Custom:STD_DDW_DIP20
Changed lines of the file:
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@@
 		(on_board yes)
 		(dnp no)
-		(property "Reference" "U24"
+		(property "Reference" "U25"
 			(at 175.26 55.88 0)
 			(effects
@@
 			)
 		)
-		(property "Footprint" "Package_DIP:DIP-20_W7.62mm_Socket_LongPads"
+		(property "Footprint" "Custom:STD_DDW_DIP20"
 			(at 172.72 71.12 0)
 			(effects
@@
 			(project "6x0x-6U"
 				(path "/d94f9d60-5ece-4752-b49c-b0d1c95f35bc/00000000-0000-0000-0000-0000526d5517"
-					(reference "U24")
+					(reference "U25")
 					(unit 1)
 				)
@@
 			)
 		)
-		(property "Footprint" "Resistor_THT:R_Array_SIP10"
+		(property "Footprint" "Custom:STD_DDW_SIP10"
 			(at 293.37 50.165 90)
 			(effects
@@
 			)
 		)
-		(property "Footprint" "Package_DIP:DIP-14_W7.62mm_Socket_LongPads"
+		(property "Footprint" "Custom:STD_DDW_DIP14"
 			(at 66.04 71.12 0)
 			(effects
@@
 			)
 		)
-		(property "Footprint" "Package_DIP:DIP-14_W7.62mm_Socket_LongPads"
+		(property "Footprint" "Custom:STD_DDW_DIP14"
 			(at 107.95 81.28 0)
 			(effects
@@
 			)
 		)
-		(property "Footprint" "Package_DIP:DIP-14_W7.62mm_Socket_LongPads"
+		(property "Footprint" "Custom:STD_DDW_DIP14"
 			(at 66.04 91.44 0)
 			(effects
@@
 		(on_board yes)
 		(dnp no)
-		(property "Reference" "U25"
+		(property "Reference" "U26"
 			(at 288.544 76.962 0)
 			(effects
@@
 			)
 		)
-		(property "Footprint" "Package_DIP:DIP-20_W7.62mm_Socket_LongPads"
+		(property "Footprint" "Custom:STD_DDW_DIP20"
 			(at 289.56 81.28 0)
 			(effects
@@
 			(project "6x0x-6U"
 				(path "/d94f9d60-5ece-4752-b49c-b0d1c95f35bc/00000000-0000-0000-0000-0000526d5517"
-					(reference "U25")
+					(reference "U26")
 					(unit 1)
 				)
@@
 		(on_board yes)
 		(dnp no)
-		(property "Reference" "U26"
+		(property "Reference" "U27"
 			(at 287.782 126.238 0)
 			(effects
@@
 			)
 		)
-		(property "Footprint" "Package_DIP:DIP-20_W7.62mm_Socket_LongPads"
+		(property "Footprint" "Custom:STD_DDW_DIP20"
 			(at 289.56 132.08 0)
 			(effects
@@
 			(project "6x0x-6U"
 				(path "/d94f9d60-5ece-4752-b49c-b0d1c95f35bc/00000000-0000-0000-0000-0000526d5517"
-					(reference "U26")
+					(reference "U27")
 					(unit 1)
 				)
@@
 		(on_board yes)
 		(dnp no)
-		(property "Reference" "U27"
+		(property "Reference" "U28"
 			(at 288.036 185.166 0)
 			(effects
@@
 			)
 		)
-		(property "Footprint" "Package_DIP:DIP-20_W7.62mm_Socket_LongPads"
+		(property "Footprint" "Custom:STD_DDW_DIP20"
 			(at 289.56 191.77 0)
 			(effects
@@
 			(project "6x0x-6U"
 				(path "/d94f9d60-5ece-4752-b49c-b0d1c95f35bc/00000000-0000-0000-0000-0000526d5517"
-					(reference "U27")
+					(reference "U28")
 					(unit 1)
 				)
@@
 		(on_board yes)
 		(dnp no)
-		(property "Reference" "#PWR055"
+		(property "Reference" "#PWR093"
 			(at 266.7 96.52 0)
 			(effects
@@
 			(project "6x0x-6U"
 				(path "/d94f9d60-5ece-4752-b49c-b0d1c95f35bc/00000000-0000-0000-0000-0000526d5517"
-					(reference "#PWR055")
+					(reference "#PWR093")
 					(unit 1)
 				)
@@
 		(on_board yes)
 		(dnp no)
-		(property "Reference" "#PWR056"
+		(property "Reference" "#PWR094"
 			(at 266.7 147.32 0)
 			(effects
@@
 			(project "6x0x-6U"
 				(path "/d94f9d60-5ece-4752-b49c-b0d1c95f35bc/00000000-0000-0000-0000-0000526d5517"
-					(reference "#PWR056")
+					(reference "#PWR094")
 					(unit 1)
 				)
@@
 		(on_board yes)
 		(dnp no)
-		(property "Reference" "#PWR057"
+		(property "Reference" "#PWR095"
 			(at 266.7 207.01 0)
 			(effects
@@
 			(project "6x0x-6U"
 				(path "/d94f9d60-5ece-4752-b49c-b0d1c95f35bc/00000000-0000-0000-0000-0000526d5517"
-					(reference "#PWR057")
+					(reference "#PWR095")
 					(unit 1)
 				)
@@
 		(on_board yes)
 		(dnp no)
-		(property "Reference" "#PWR053"
+		(property "Reference" "#PWR091"
 			(at 172.72 48.26 0)
 			(effects
@@
 			(project "6809PC-6U"
 				(path "/d94f9d60-5ece-4752-b49c-b0d1c95f35bc/00000000-0000-0000-0000-0000526d5517"
-					(reference "#PWR053")
+					(reference "#PWR091")
 					(unit 1)
 				)
@@
 		(on_board yes)
 		(dnp no)
-		(property "Reference" "P9"
+		(property "Reference" "P13"
 			(at 52.832 131.826 0)
 			(effects
@@
 			)
 		)
-		(property "Footprint" "Package_DIP:DIP-14_W7.62mm_Socket_LongPads"
+		(property "Footprint" "Custom:STD_DDW_DIP14"
 			(at 53.34 132.08 0)
 			(effects
@@
 			(project "6809PC-6U"
 				(path "/d94f9d60-5ece-4752-b49c-b0d1c95f35bc/00000000-0000-0000-0000-0000526d5517"
-					(reference "P9")
+					(reference "P13")
 					(unit 1)
 				)
@@
 			)
 		)
-		(property "Footprint" "Package_DIP:DIP-14_W7.62mm_Socket_LongPads"
+		(property "Footprint" "Custom:STD_DDW_DIP14"
 			(at 137.16 171.45 0)
 			(effects
@@
 		(on_board yes)
 		(dnp no)
-		(property "Reference" "#PWR050"
+		(property "Reference" "#PWR088"
 			(at 46.99 153.67 0)
 			(effects
@@
 			(project "6809PC-6U"
 				(path "/d94f9d60-5ece-4752-b49c-b0d1c95f35bc/00000000-0000-0000-0000-0000526d5517"
-					(reference "#PWR050")
+					(reference "#PWR088")
 					(unit 1)
 				)
@@
 			)
 		)
-		(property "Footprint" "Package_DIP:DIP-14_W7.62mm_Socket_LongPads"
+		(property "Footprint" "Custom:STD_DDW_DIP14"
 			(at 138.43 199.39 0)
 			(effects
@@
 		(on_board yes)
 		(dnp no)
-		(property "Reference" "#PWR051"
+		(property "Reference" "#PWR089"
 			(at 59.69 132.08 0)
 			(effects
@@
 			(project "6809PC-6U"
 				(path "/d94f9d60-5ece-4752-b49c-b0d1c95f35bc/00000000-0000-0000-0000-0000526d5517"
-					(reference "#PWR051")
+					(reference "#PWR089")
 					(unit 1)
 				)
@@
 		(on_board yes)
 		(dnp no)
-		(property "Reference" "#PWR058"
+		(property "Reference" "#PWR096"
 			(at 289.56 58.42 0)
 			(effects
@@
 			(project "6809PC-6U"
 				(path "/d94f9d60-5ece-4752-b49c-b0d1c95f35bc/00000000-0000-0000-0000-0000526d5517"
-					(reference "#PWR058")
+					(reference "#PWR096")
 					(unit 1)
 				)
@@
 			)
 		)
-		(property "Footprint" "Package_DIP:DIP-14_W7.62mm_Socket_LongPads"
+		(property "Footprint" "Custom:STD_DDW_DIP14"
 			(at 137.16 154.94 0)
 			(effects
@@
 		(on_board yes)
 		(dnp no)
-		(property "Reference" "#PWR054"
+		(property "Reference" "#PWR092"
 			(at 172.72 91.44 0)
 			(effects
@@
 			(project "6809PC-6U"
 				(path "/d94f9d60-5ece-4752-b49c-b0d1c95f35bc/00000000-0000-0000-0000-0000526d5517"
-					(reference "#PWR054")
+					(reference "#PWR092")
 					(unit 1)
 				)
@@
 		(on_board yes)
 		(dnp no)
-		(property "Reference" "#PWR061"
+		(property "Reference" "#PWR099"
 			(at 289.56 152.4 0)
 			(effects
@@
 			(project "6809PC-6U"
 				(path "/d94f9d60-5ece-4752-b49c-b0d1c95f35bc/00000000-0000-0000-0000-0000526d5517"
-					(reference "#PWR061")
+					(reference "#PWR099")
 					(unit 1)
 				)
@@
 		(on_board yes)
 		(dnp no)
-		(property "Reference" "#PWR059"
+		(property "Reference" "#PWR097"
 			(at 289.56 101.6 0)
 			(effects
@@
 			(project "6809PC-6U"
 				(path "/d94f9d60-5ece-4752-b49c-b0d1c95f35bc/00000000-0000-0000-0000-0000526d5517"
-					(reference "#PWR059")
+					(reference "#PWR097")
 					(unit 1)
 				)
@@
 			)
 		)
-		(property "Footprint" "Capacitor_THT:C_Disc_D5.0mm_W2.5mm_P5.00mm"
+		(property "Footprint" "Custom:STD_DDW_CAP"
 			(at 65.7352 142.24 0)
 			(effects
@@
 			)
 		)
-		(property "Footprint" "Package_DIP:DIP-14_W7.62mm_Socket_LongPads"
+		(property "Footprint" "Custom:STD_DDW_DIP14"
 			(at 134.62 123.19 0)
 			(effects
@@
 			)
 		)
-		(property "Footprint" "Package_DIP:DIP-14_W7.62mm_Socket_LongPads"
+		(property "Footprint" "Custom:STD_DDW_DIP14"
 			(at 135.89 139.7 0)
 			(effects
@@
 			)
 		)
-		(property "Footprint" "Package_DIP:DIP-14_W7.62mm_Socket_LongPads"
+		(property "Footprint" "Custom:STD_DDW_DIP14"
 			(at 137.16 186.69 0)
 			(effects
@@
 		(on_board yes)
 		(dnp no)
-		(property "Reference" "#PWR060"
+		(property "Reference" "#PWR098"
 			(at 289.56 109.22 0)
 			(effects
@@
 			(project "6809PC-6U"
 				(path "/d94f9d60-5ece-4752-b49c-b0d1c95f35bc/00000000-0000-0000-0000-0000526d5517"
-					(reference "#PWR060")
+					(reference "#PWR098")
 					(unit 1)
 				)
@@
 		(on_board yes)
 		(dnp no)
-		(property "Reference" "#PWR052"
+		(property "Reference" "#PWR090"
 			(at 64.77 142.24 0)
 			(effects
@@
 			(project "6809PC-6U"
 				(path "/d94f9d60-5ece-4752-b49c-b0d1c95f35bc/00000000-0000-0000-0000-0000526d5517"
-					(reference "#PWR052")
+					(reference "#PWR090")
 					(unit 1)
 				)
@@
 		(on_board yes)
 		(dnp no)
-		(property "Reference" "#PWR063"
+		(property "Reference" "#PWR0101"
 			(at 289.56 212.09 0)
 			(effects
@@
 			(project "6809PC-6U"
 				(path "/d94f9d60-5ece-4752-b49c-b0d1c95f35bc/00000000-0000-0000-0000-0000526d5517"
-					(reference "#PWR063")
+					(reference "#PWR0101")
 					(unit 1)
 				)
@@
 		(on_board yes)
 		(dnp no)
-		(property "Reference" "#PWR062"
+		(property "Reference" "#PWR0100"
 			(at 289.56 168.91 0)
 			(effects
@@
 			(project "6809PC-6U"
 				(path "/d94f9d60-5ece-4752-b49c-b0d1c95f35bc/00000000-0000-0000-0000-0000526d5517"
-					(reference "#PWR062")
+					(reference "#PWR0100")
 					(unit 1)
 				)

Commit message: V1.1
Parts:
- added R26: 4.7K, Custom:STD_DDW_RESISTOR, symbol Device:R
Connections:
- net B_INT: now also R26.1
- net GND: now also R26.2
Other:
- note removed: "rev. 011: /RESET and /B_NMI added to RR6 pull-ups"
Changed lines of the file:
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@@
 	(wire
 		(pts
+			(xy 336.55 25.4) (xy 336.55 24.13)
+		)
+		(stroke
+			(width 0)
+			(type default)
+		)
+	)
+	(wire
+		(pts
 			(xy 309.88 81.28) (xy 302.26 81.28)
 		)
@@
 	(wire
 		(pts
+			(xy 336.55 24.13) (xy 335.28 24.13)
+		)
+		(stroke
+			(width 0)
+			(type default)
+		)
+	)
+	(wire
+		(pts
 			(xy 255.27 196.85) (xy 276.86 196.85)
 		)
@@
 	(wire
 		(pts
+			(xy 325.12 24.13) (xy 327.66 24.13)
+		)
+		(stroke
+			(width 0)
+			(type default)
+		)
+	)
+	(wire
+		(pts
 			(xy 265.43 124.46) (xy 276.86 124.46)
 		)
@@
 		)
 	)
-	(text "rev. 011:  /RESET and /B_NMI added\nto RR6 pull-ups"
-		(exclude_from_sim no)
-		(at 262.89 52.07 0)
-		(effects
-			(font
-				(size 1.524 1.524)
-			)
-			(justify left bottom)
-		)
-	)
 	(label "GND"
 		(at 149.86 83.82 0)
@@
 		)
 	)
+	(global_label "B_INT"
+		(shape input)
+		(at 325.12 24.13 180)
+		(fields_autoplaced yes)
+		(effects
+			(font
+				(size 1.27 1.27)
+			)
+			(justify right)
+		)
+		(property "Intersheetrefs" "${INTERSHEET_REFS}"
+			(at 317.6485 24.13 0)
+			(effects
+				(font
+					(size 1.27 1.27)
+				)
+				(justify right)
+				(hide yes)
+			)
+		)
+	)
 	(global_label "B_A8"
 		(shape bidirectional)
@@
 	)
 	(symbol
+		(lib_id "Device:R")
+		(at 331.47 24.13 90)
+		(unit 1)
+		(exclude_from_sim no)
+		(in_bom yes)
+		(on_board yes)
+		(dnp no)
+		(property "Reference" "R26"
+			(at 331.47 22.098 90)
+			(effects
+				(font
+					(size 1.27 1.27)
+				)
+			)
+		)
+		(property "Value" "4.7K"
+			(at 331.47 24.13 90)
+			(effects
+				(font
+					(size 1.27 1.27)
+				)
+			)
+		)
+		(property "Footprint" "Custom:STD_DDW_RESISTOR"
+			(at 331.47 25.908 90)
+			(effects
+				(font
+					(size 1.27 1.27)
+				)
+				(hide yes)
+			)
+		)
+		(property "Datasheet" "~"
+			(at 331.47 24.13 0)
+			(effects
+				(font
+					(size 1.27 1.27)
+				)
+				(hide yes)
+			)
+		)
+		(property "Description" "Resistor"
+			(at 331.47 24.13 0)
+			(effects
+				(font
+					(size 1.27 1.27)
+				)
+				(hide yes)
+			)
+		)
+		(pin "1"
+		)
+		(pin "2"
+		)
+		(instances
+			(project "6809PC-6U"
+				(path "/d94f9d60-5ece-4752-b49c-b0d1c95f35bc/00000000-0000-0000-0000-0000526d5517"
+					(reference "R26")
+					(unit 1)
+				)
+			)
+		)
+	)
+	(symbol
 		(lib_id "power:VCC")
 		(at 289.56 60.96 0)
@@
 					(unit 1)
 				)
+			)
+		)
+	)
+	(symbol
+		(lib_id "power:GND")
+		(at 336.55 25.4 0)
+		(unit 1)
+		(exclude_from_sim no)
+		(in_bom yes)
+		(on_board yes)
+		(dnp no)
+		(property "Reference" "#PWR0211"
+			(at 336.55 25.4 0)
+			(effects
+				(font
+					(size 0.762 0.762)
+				)
+				(hide yes)
+			)
+		)
+		(property "Value" "GND"
+			(at 336.55 27.178 0)
+			(effects
+				(font
+					(size 0.762 0.762)
+				)
+				(hide yes)
+			)
+		)
+		(property "Footprint" ""
+			(at 336.55 25.4 0)
+			(effects
+				(font
+					(size 1.27 1.27)
+				)
+				(hide yes)
+			)
+		)
+		(property "Datasheet" ""
+			(at 336.55 25.4 0)
+			(effects
+				(font
+					(size 1.27 1.27)
+				)
+				(hide yes)
+			)
+		)
+		(property "Description" "Power symbol creates a global label with name \"GND\" , ground"
+			(at 336.55 25.4 0)
+			(effects
+				(font
+					(size 1.27 1.27)
+				)
+				(hide yes)
+			)
+		)
+		(pin "1"
+		)
+		(instances
+			(project "6809PC-6U"
+				(path "/d94f9d60-5ece-4752-b49c-b0d1c95f35bc/00000000-0000-0000-0000-0000526d5517"
+					(reference "#PWR0211")
+					(unit 1)
+				)

Commit message: 6809PC work
Connections:
- net PULLUP4: no longer names the net of RR1.7 (R6)
- no-connect marks 8 -> 9
Changed lines of the file:
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@@
 	(title_block
 		(title "6809PC")
-		(date "2025-01-21")
-		(rev "001")
+		(date "2025-05-17")
+		(rev "002")
 		(comment 1 "https://github.com/danwerner21/6809PC")
 		(comment 2 "Based on work by Andrew Lynch and John Coffman")
@@
 	)
 	(no_connect
+		(at 279.4 38.1)
+	)
+	(no_connect
 		(at 59.69 139.7)
 	)
@@
 		)
 	)
-	(global_label "PULLUP4"
-		(shape input)
-		(at 279.4 38.1 180)
-		(fields_autoplaced yes)
-		(effects
-			(font
-				(size 1.27 1.27)
-			)
-			(justify right)
-		)
-		(property "Intersheetrefs" "${INTERSHEET_REFS}"
-			(at 268.6023 38.1 0)
-			(effects
-				(font
-					(size 1.27 1.27)
-				)
-				(justify right)
-				(hide yes)
-			)
-		)
-	)
 	(global_label "B_A15"
 		(shape tri_state)
@@
 					(size 1.27 1.27)
 				)
+				(hide yes)
+			)
+		)
+	)
+	(global_label "PULLUP3"
+		(shape input)
+		(at 279.4 33.02 180)
+		(fields_autoplaced yes)
+		(effects
+			(font
+				(size 1.27 1.27)
+			)
+			(justify right)
+		)
+		(property "Intersheetrefs" "${INTERSHEET_REFS}"
+			(at 268.6023 33.02 0)
+			(effects
+				(font
+					(size 1.27 1.27)
+				)
+				(justify right)
 				(hide yes)
 			)
@@
 				(hide yes)
 			)
-		)
-	)
-	(global_label "PULLUP3"
-		(shape input)
-		(at 279.4 33.02 180)
-		(fields_autoplaced yes)
-		(effects
-			(font
-				(size 1.27 1.27)
-			)
-			(justify right)
-		)
-		(property "Intersheetrefs" "${INTERSHEET_REFS}"
-			(at 268.6023 33.02 0)
-			(effects
-				(font
-					(size 1.27 1.27)
-				)
-				(justify right)
-				(hide yes)
-			)
