File: MMU-4.kicad_sch (KiCad schematic)
At the start: 15 parts, among them U1 74LS04, U20 74LS74, U29 74LS08, U30 74LS174, U31 74LS244, U32 74LS157, U33 74LS374, U34 74LS244, U35 SRAM-32K, U36 74LS245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

Commit message: Schematic in progress
Parts:
- U1: footprint DIP-14__300 -> Package_DIP:DIP-14_W7.62mm_Socket_LongPads
- U15: renamed from U29; footprint DIP-14__300 -> Package_DIP:DIP-14_W7.62mm_Socket_LongPads
- U22: renamed from U20; footprint DIP-14__300 -> Package_DIP:DIP-14_W7.62mm_Socket_LongPads
- U34: renamed from U30; footprint DIP-16__300 -> Package_DIP:DIP-16_W7.62mm_Socket_LongPads
- U35: renamed from U31; footprint DIP-20__300 -> Package_DIP:DIP-20_W7.62mm_Socket_LongPads
- U36: renamed from U32; footprint DIP-16__300 -> Package_DIP:DIP-16_W7.62mm_Socket_LongPads
- U37: renamed from U33; footprint DIP-20__300 -> Package_DIP:DIP-20_W7.62mm_Socket_LongPads
- U38: renamed from U34; footprint DIP-20__300 -> Package_DIP:DIP-20_W7.62mm_Socket_LongPads
- U39: renamed from U35; footprint Package_DIP:DIP-28_W15.24mm -> Package_DIP:DIP-28_W7.62mm_Socket_LongPads
- U40: renamed from U36; footprint DIP-20__300 -> Package_DIP:DIP-20_W7.62mm_Socket_LongPads
- U41: renamed from U37; footprint DIP-16__300 -> Package_DIP:DIP-16_W7.62mm_Socket_LongPads
- U42: renamed from U38; footprint DIP-16__300 -> Package_DIP:DIP-16_W7.62mm_Socket_LongPads
- U43: renamed from U39; footprint DIP-16__300 -> Package_DIP:DIP-16_W7.62mm_Socket_LongPads
- U44: renamed from U40; footprint DIP-20__300 -> Package_DIP:DIP-20_W7.62mm_Socket_LongPads
- U45: renamed from U41; footprint DIP-20__300 -> Package_DIP:DIP-20_W7.62mm_Socket_LongPads
Connections:
- net /MMU-ENB-WR: now also U22.11 (C); no longer U22.3 (C)
- net MMU-ENABLE: now also U22.9 (Q); no longer U22.5 (Q)
- net VCC: now also U22.10 (~{S}), U43.16 (VCC); no longer U22.4 (~{S})
- net mD0: now also U22.12 (D); no longer U22.2 (D)
- net at U15.6: now also U22.13 (~{R}); no longer U22.1 (~{R})
Other:
- company: N8VEM Users Group -> (none)
- title: 6809 and 6502 ATX and 6U -> 6809PC

Commit message: PCB in progress
Parts:
- removed unit 4 of U15
- added U10: 74LS32, Custom:STD_DDW_DIP14, symbol 74xx:74LS32
- U1, U15, U22: footprint Package_DIP:DIP-14_W7.62mm_Socket_LongPads -> Custom:STD_DDW_DIP14
- U35: renamed from U34; footprint Package_DIP:DIP-16_W7.62mm_Socket_LongPads -> Custom:STD_DDW_DIP16
- U36: renamed from U35; footprint Package_DIP:DIP-20_W7.62mm_Socket_LongPads -> Custom:STD_DDW_DIP20
- U37: renamed from U36; footprint Package_DIP:DIP-16_W7.62mm_Socket_LongPads -> Custom:STD_DDW_DIP16
- U38: renamed from U37; footprint Package_DIP:DIP-20_W7.62mm_Socket_LongPads -> Custom:STD_DDW_DIP20
- U39: renamed from U38; footprint Package_DIP:DIP-20_W7.62mm_Socket_LongPads -> Custom:STD_DDW_DIP20
- U40: renamed from U39; footprint Package_DIP:DIP-28_W7.62mm_Socket_LongPads -> Custom:STD_DDW_DIP28_SKINNY
- U41: renamed from U40; footprint Package_DIP:DIP-20_W7.62mm_Socket_LongPads -> Custom:STD_DDW_DIP20
- U42: renamed from U41; footprint Package_DIP:DIP-16_W7.62mm_Socket_LongPads -> Custom:STD_DDW_DIP16
- U43: renamed from U42; footprint Package_DIP:DIP-16_W7.62mm_Socket_LongPads -> Custom:STD_DDW_DIP16
- U44: renamed from U43; footprint Package_DIP:DIP-16_W7.62mm_Socket_LongPads -> Custom:STD_DDW_DIP16
- U45: renamed from U44; footprint Package_DIP:DIP-20_W7.62mm_Socket_LongPads -> Custom:STD_DDW_DIP20
- U46: renamed from U45; footprint Package_DIP:DIP-20_W7.62mm_Socket_LongPads -> Custom:STD_DDW_DIP20
Connections:
- net /MMU-ENB-WR: now also U42.13 (O2); no longer U42.12 (O3)
- net /MMU-MAP-RD: now also U10.11; no longer U42.9 (O6)
- net /MMU-MAP-WR: now also U10.8; no longer U42.13 (O2)
- net mA0: now also U42.1 (A0)
- net mA1: now also U42.2 (A1)
- net mA4: no longer U42.1 (A0)
- net mA5: no longer U42.2 (A1)
- net /IOSEL-0EAxx renamed /IOSEL-0EFE0
- net /MMU-MAP-RW renamed /IOSEL-0EFD0
- net /IOSEL-0EFD0: now also U10.10, U10.12
- new net CPU_/RD: U10.13
- new net CPU_/WR: U10.9
- no-connect marks 13 -> 15

Commit message: V1.1
Connections:
- net GND: now also U42.8 (GND); no longer U42.16 (VCC)
- net VCC: now also U42.16 (VCC); no longer U42.8 (GND)
- net TC: now reaches U42.9 (O6)
- no-connect marks 15 -> 14
Other:
- note added: "Patch from V1.0 to V1.1 * Connect U42 pin 9 to Slots pin 27 * LS138 U42 and U24 have miswired power * U24 Pin 6 should be VCC not GND"
Changed lines of the file:
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@@
 	)
 	(no_connect
-		(at 242.57 220.98)
-	)
-	(no_connect
 		(at 128.27 123.19)
 	)
@@
 	(wire
 		(pts
+			(xy 229.87 210.82) (xy 229.87 208.28)
+		)
+		(stroke
+			(width 0)
+			(type default)
+		)
+	)
+	(wire
+		(pts
 			(xy 200.66 95.25) (xy 208.28 95.25)
 		)
@@
 	(wire
 		(pts
+			(xy 229.87 243.84) (xy 241.3 243.84)
+		)
+		(stroke
+			(width 0)
+			(type default)
+		)
+	)
+	(wire
+		(pts
 			(xy 167.64 69.85) (xy 167.64 77.47)
 		)
@@
 	(wire
 		(pts
+			(xy 229.87 208.28) (xy 232.41 208.28)
+		)
+		(stroke
+			(width 0)
+			(type default)
+		)
+	)
+	(wire
+		(pts
 			(xy 135.89 85.09) (xy 135.89 107.95)
 		)
@@
 	(wire
 		(pts
+			(xy 242.57 220.98) (xy 246.38 220.98)
+		)
+		(stroke
+			(width 0)
+			(type default)
+		)
+	)
+	(wire
+		(pts
 			(xy 200.66 82.55) (xy 213.36 82.55)
 		)
@@
 		)
 	)
+	(text "Patch from V1.0 to V1.1\n* Connect U42 pin 9 to Slots pin 27 \n* LS138 U42 and U24 have miswired power\n* U24 Pin 6 should be VCC not GND"
+		(exclude_from_sim no)
+		(at 304.546 225.044 0)
+		(effects
+			(font
+				(size 2 2)
+				(thickness 0.4)
+				(bold yes)
+			)
+			(justify left)
+		)
+	)
 	(text "SRAM - skinny 28-pin DIP\n35ns 8K or 32K; e.g.,\nany Cypress or JEDEC\npart."
 		(exclude_from_sim no)
@@
 	)
 	(label "/MMU-MAP-RW"
-		(at 158.75 248.92 180)
+		(at 157.48 248.92 180)
 		(fields_autoplaced yes)
 		(effects
@@
 		)
 	)
+	(global_label "TC"
+		(shape output)
+		(at 246.38 220.98 0)
+		(fields_autoplaced yes)
+		(effects
+			(font
+				(size 1.27 1.27)
+			)
+			(justify left)
+		)
+		(property "Intersheetrefs" "${INTERSHEET_REFS}"
+			(at 250.9486 220.98 0)
+			(effects
+				(font
+					(size 1.27 1.27)
+				)
+				(justify left)
+				(hide yes)
+			)
+		)
+	)
 	(global_label "LA5"
 		(shape input)
@@
 		(dnp no)
 		(property "Reference" "U45"
-			(at 372.11 39.37 0)
+			(at 370.586 39.878 0)
 			(effects
 				(font
@@
 	(symbol
 		(lib_id "power:VCC")
-		(at 229.87 210.82 0)
+		(at 241.3 243.84 0)
 		(unit 1)
 		(exclude_from_sim no)
@@
 		(dnp no)
 		(property "Reference" "#PWR0136"
-			(at 229.87 208.28 0)
+			(at 241.3 241.3 0)
 			(effects
 				(font
@@
 		)
 		(property "Value" "VCC"
-			(at 229.87 208.28 0)
+			(at 241.3 241.3 0)
 			(effects
 				(font
@@
 		)
 		(property "Footprint" ""
-			(at 229.87 210.82 0)
+			(at 241.3 243.84 0)
 			(effects
 				(font
@@
 		)
 		(property "Datasheet" ""
-			(at 229.87 210.82 0)
+			(at 241.3 243.84 0)
 			(effects
 				(font
@@
 		)
 		(property "Description" "Power symbol creates a global label with name \"VCC\""
-			(at 229.87 210.82 0)
+			(at 241.3 243.84 0)
 			(effects
 				(font
@@
 	(symbol
 		(lib_id "power:GND")
-		(at 229.87 243.84 0)
+		(at 232.41 208.28 0)
 		(unit 1)
 		(exclude_from_sim no)
@@
 		(dnp no)
 		(property "Reference" "#PWR0137"
-			(at 229.87 243.84 0)
+			(at 232.41 208.28 0)
 			(effects
 				(font
@@
 		)
 		(property "Value" "GND"
-			(at 229.87 245.618 0)
+			(at 232.41 210.058 0)
 			(effects
 				(font
@@
 		)
 		(property "Footprint" ""
-			(at 229.87 243.84 0)
+			(at 232.41 208.28 0)
 			(effects
 				(font
@@
 		)
 		(property "Datasheet" ""
-			(at 229.87 243.84 0)
+			(at 232.41 208.28 0)
 			(effects
 				(font
@@
 		)
 		(property "Description" "Power symbol creates a global label with name \"GND\" , ground"
-			(at 229.87 243.84 0)
+			(at 232.41 208.28 0)
 			(effects
 				(font

Commit message: 6809PC work
Connections:
- net mA6: no longer U42.5 (E2)
- net /IOSEL-0EFE0: now also U42.5 (E2)
Changed lines of the file:
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@@
 	(title_block
 		(title "6809PC")
-		(date "2025-01-21")
-		(rev "001")
+		(date "2025-05-17")
+		(rev "002")
 		(comment 1 "https://github.com/danwerner21/6809PC")
 		(comment 2 "Based on work by Andrew Lynch and John Coffman")
@@
 	)
 	(junction
+		(at 213.36 218.44)
+		(diameter 0)
+		(color 0 0 0 0)
+	)
+	(junction
 		(at 175.26 100.33)
 		(diameter 0)
@@
 	(wire
 		(pts
-			(xy 217.17 218.44) (xy 212.09 218.44)
+			(xy 217.17 218.44) (xy 213.36 218.44)
 		)
 		(stroke
@@
 	(wire
 		(pts
-			(xy 190.5 220.98) (xy 217.17 220.98)
-		)
-		(stroke
-			(width 0)
-			(type default)
-		)
-	)
-	(wire
-		(pts
 			(xy 229.87 210.82) (xy 229.87 208.28)
 		)
@@
 	(wire
 		(pts
+			(xy 217.17 220.98) (xy 213.36 220.98)
+		)
+		(stroke
+			(width 0)
+			(type default)
+		)
+	)
+	(wire
+		(pts
 			(xy 81.28 154.94) (xy 106.68 154.94)
 		)
@@
 	(wire
 		(pts
+			(xy 213.36 218.44) (xy 213.36 220.98)
+		)
+		(stroke
+			(width 0)
+			(type default)
+		)
+	)
+	(wire
+		(pts
 			(xy 255.27 86.36) (xy 314.96 86.36)
 		)
@@
 	(wire
 		(pts
+			(xy 213.36 218.44) (xy 212.09 218.44)
+		)
+		(stroke
+			(width 0)
+			(type default)
+		)
+	)
+	(wire
+		(pts
 			(xy 124.46 237.49) (xy 128.27 237.49)
 		)
@@
 			(effects
 				(font
-					(size 1.27 1.27)
-				)
-				(hide yes)
-			)
-		)
-	)
-	(global_label "mA6"
-		(shape input)
-		(at 190.5 220.98 180)
-		(effects
-			(font
-				(size 1.524 1.524)
-			)
-			(justify right)
-		)
-		(property "Intersheetrefs" "${INTERSHEET_REFS}"
-			(at 190.5 220.98 0)
-			(effects
-				(font
