File: RTC.kicad_sch (KiCad schematic)
At the start: 4 parts, among them P12 CONN_4, U42 DS1302, X1 RTC_OSC

Commit message: Schematic in progress
Parts:
- removed JP3: JUMPER, PIN_ARRAY_2X1, symbol Jumper:Jumper_2_Open
- removed U42: DS1302, Package_DIP:DIP-8_W7.62mm, symbol Timer_RTC:DS1302+
- added C59, C60: 15pf, Capacitor_THT:C_Disc_D5.0mm_W2.5mm_P5.00mm, symbol Device:C
- added D3, D4: D, Diode_THT:D_DO-41_SOD81_P10.16mm_Horizontal, symbol Device:D
- added U46: ~, Package_DIP:DIP-18_W7.62mm_Socket_LongPads, symbol Custom:M6242B
- P12: footprint PIN_ARRAY_4x1 -> Connector_PinHeader_2.54mm:PinHeader_1x04_P2.54mm_Vertical
- X1: footprint C1 -> Crystal:Crystal_DS10_D1.0mm_L4.3mm_Horizontal
Connections:
- net GND: now also U46.9 (GND)
- net VCC: now also D3.2 (A)
- net at X1.2: now also C59.2, U46.17 (XT1)
- net at X1.1: now also C60.2, U46.16 (XT)
- net at P12.1 (Pin_1): now also D4.2 (A)
- new net: C59.1, C60.1, D3.1 (K), D4.1 (K), U46.18 (VCC)
- new net /IOSEL-0EExx: U46.2 (CS0)
- new net BUSALE: U46.3 (ALE)
- new net CPU_/RD: U46.8 (RD)
- new net CPU_/WR: U46.10 (WR)
- new net PULLUP1: U46.15 (CS1)
- new net mA0: U46.4 (A0)
- new net mA1: U46.5 (A1)
- new net mA2: U46.6 (A2)
- new net mA3: U46.7 (A3)
- new net mD0: U46.14 (D0)
- new net mD1: U46.13 (D1)
- new net mD2: U46.12 (D2)
- new net mD3: U46.11 (D3)
- no-connect marks 0 -> 1
Other:
- company: N8VEM Users Group -> (none)
- title: 6809 and 6502 ATX and 6U -> 6809PC
- moved on the sheet: X1

Commit message: PCB in progress
Parts:
- C59, C60: footprint Capacitor_THT:C_Disc_D5.0mm_W2.5mm_P5.00mm -> Custom:STD_DDW_CAP
- D3, D4: footprint Diode_THT:D_DO-41_SOD81_P10.16mm_Horizontal -> Custom:STD_DDW_DIODE
- P16: renamed from P12; footprint Connector_PinHeader_2.54mm:PinHeader_1x04_P2.54mm_Vertical -> Custom:STD_DDW_PINHEAD_V_1x04
- U47: renamed from U46; footprint Package_DIP:DIP-18_W7.62mm_Socket_LongPads -> Custom:STD_DDW_DIP18
- X1: footprint Crystal:Crystal_DS10_D1.0mm_L4.3mm_Horizontal -> Custom:DDW_STD_RTCCRYSTAL
Connections:
- net /IOSEL-0EExx renamed /IOSEL-0EF90
Changed lines of the file:
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@@
 		)
 	)
-	(global_label "/IOSEL-0EExx"
-		(shape output)
+	(global_label "{slash}IOSEL-0EF90"
+		(shape input)
 		(at 88.9 120.65 180)
 		(effects
@@
 		(on_board yes)
 		(dnp no)
-		(property "Reference" "#PWR0110"
+		(property "Reference" "#PWR0148"
 			(at 109.22 92.71 0)
 			(effects
@@
 			(project "6x0x-6U"
 				(path "/d94f9d60-5ece-4752-b49c-b0d1c95f35bc/00000000-0000-0000-0000-00005274ff2a"
-					(reference "#PWR0110")
+					(reference "#PWR0148")
 					(unit 1)
 				)
@@
 			)
 		)
-		(property "Footprint" "Crystal:Crystal_DS10_D1.0mm_L4.3mm_Horizontal"
+		(property "Footprint" "Custom:DDW_STD_RTCCRYSTAL"
 			(at 133.35 116.84 0)
 			(effects
@@
 		(on_board yes)
 		(dnp no)
-		(property "Reference" "P12"
+		(property "Reference" "P16"
 			(at 166.37 91.694 90)
 			(effects
@@
 			)
 		)
-		(property "Footprint" "Connector_PinHeader_2.54mm:PinHeader_1x04_P2.54mm_Vertical"
+		(property "Footprint" "Custom:STD_DDW_PINHEAD_V_1x04"
 			(at 166.37 97.79 0)
 			(effects
@@
 			(project "6x0x-6U"
 				(path "/d94f9d60-5ece-4752-b49c-b0d1c95f35bc/00000000-0000-0000-0000-00005274ff2a"
-					(reference "P12")
+					(reference "P16")
 					(unit 1)
 				)
@@
 		(on_board yes)
 		(dnp no)
-		(property "Reference" "#PWR0112"
+		(property "Reference" "#PWR0150"
 			(at 158.75 105.41 0)
 			(effects
@@
 			(project "6x0x-6U"
 				(path "/d94f9d60-5ece-4752-b49c-b0d1c95f35bc/00000000-0000-0000-0000-00005274ff2a"
-					(reference "#PWR0112")
+					(reference "#PWR0150")
 					(unit 1)
 				)
@@
 			)
 		)
-		(property "Footprint" "Diode_THT:D_DO-41_SOD81_P10.16mm_Horizontal"
+		(property "Footprint" "Custom:STD_DDW_DIODE"
 			(at 109.22 99.06 0)
 			(effects
@@
 			)
 		)
-		(property "Footprint" "Capacitor_THT:C_Disc_D5.0mm_W2.5mm_P5.00mm"
+		(property "Footprint" "Custom:STD_DDW_CAP"
 			(at 130.5052 107.95 0)
 			(effects
@@
 		(dnp no)
 		(fields_autoplaced yes)
-		(property "Reference" "U46"
+		(property "Reference" "U47"
 			(at 111.4141 111.76 0)
 			(effects
@@
 			)
 		)
-		(property "Footprint" "Package_DIP:DIP-18_W7.62mm_Socket_LongPads"
+		(property "Footprint" "Custom:STD_DDW_DIP18"
 			(at 109.22 121.92 0)
 			(effects
@@
 			(project ""
 				(path "/d94f9d60-5ece-4752-b49c-b0d1c95f35bc/00000000-0000-0000-0000-00005274ff2a"
-					(reference "U46")
+					(reference "U47")
 					(unit 1)
 				)
@@
 			)
 		)
-		(property "Footprint" "Capacitor_THT:C_Disc_D5.0mm_W2.5mm_P5.00mm"
+		(property "Footprint" "Custom:STD_DDW_CAP"
 			(at 138.1252 107.95 0)
 			(effects
@@
 		(on_board yes)
 		(dnp no)
-		(property "Reference" "#PWR0111"
+		(property "Reference" "#PWR0149"
 			(at 109.22 143.51 0)
 			(effects
@@
 			(project "6809PC-6U"
 				(path "/d94f9d60-5ece-4752-b49c-b0d1c95f35bc/00000000-0000-0000-0000-00005274ff2a"
-					(reference "#PWR0111")
+					(reference "#PWR0149")
 					(unit 1)
 				)
@@
 			)
 		)
-		(property "Footprint" "Diode_THT:D_DO-41_SOD81_P10.16mm_Horizontal"
+		(property "Footprint" "Custom:STD_DDW_DIODE"
 			(at 120.65 102.87 0)
 			(effects

Commit message: 6809PC work
Parts:
- U47: value ~ -> M6242
Changed lines of the file:
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@@
 	(title_block
 		(title "6809PC")
-		(date "2025-01-21")
-		(rev "001")
+		(date "2025-05-17")
+		(rev "002")
 		(comment 1 "https://github.com/danwerner21/6809PC")
 		(comment 2 "Based on work by Andrew Lynch and John Coffman")
@@
 			)
 		)
-		(property "Value" "~"
+		(property "Value" "M6242"
 			(at 111.4141 114.3 0)
 			(effects
@@
 			)
 		)
-		(property "Description" ""
+		(property "Description" "M6242"
 			(at 109.22 121.92 0)
 			(effects
