File: cpu-6809.kicad_sch (KiCad schematic)
At the start: 21 parts, among them K2 CONN_3, P10 16.000Mhz, P11 CONN_4X2, U1 74LS04, U12 74LS00, U21 74LS14, U22 74LS06, U24 74LS163, U25 74LS240, U26 74LS245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

Commit message: Schematic in progress
Parts:
- removed R5, R6: 2200, R3, symbol Device:R
- removed unit 4 of U21
- removed XK1: CONN_3X2, PIN_ARRAY_3x2, symbol 6x0x-6U-rescue:CONN_3X2
- removed XK2: CONN_3, PIN_ARRAY_3X1, symbol Connector_Generic:Conn_01x03
- C58: renamed from C57; footprint C2 -> Capacitor_THT:C_Disc_D5.0mm_W2.5mm_P5.00mm
- JP2: footprint PIN_ARRAY_2X1 -> Connector_PinHeader_2.54mm:PinHeader_1x02_P2.54mm_Vertical
- K2: footprint PIN_ARRAY_3X1 -> Connector_PinHeader_2.54mm:PinHeader_1x03_P2.54mm_Vertical
- P10, U1, U5, U6: footprint DIP-14__300 -> Package_DIP:DIP-14_W7.62mm_Socket_LongPads
- P11: footprint PIN_ARRAY_4x2 -> Connector_PinHeader_2.54mm:PinHeader_2x04_P2.54mm_Vertical
- U17: renamed from U21; footprint DIP-14__300 -> Package_DIP:DIP-14_W7.62mm_Socket_LongPads
- U18: renamed from U22; footprint DIP-14__300 -> Package_DIP:DIP-14_W7.62mm_Socket_LongPads
- U21: renamed from U12; footprint DIP-14__300 -> Package_DIP:DIP-14_W7.62mm_Socket_LongPads
- U29: renamed from U24; footprint DIP-16__300 -> Package_DIP:DIP-16_W7.62mm_Socket_LongPads
- U30: renamed from U25; footprint DIP-20__300 -> Package_DIP:DIP-20_W7.62mm_Socket_LongPads
- U31: renamed from U26; footprint DIP-20__300 -> Package_DIP:DIP-20_W7.62mm_Socket_LongPads
- U32: renamed from U27; footprint Package_DIP:DIP-40_W15.24mm -> Package_DIP:DIP-40_W15.24mm_Socket_LongPads
- U33: renamed from U28; footprint DIP-20__300 -> Package_DIP:DIP-20_W7.62mm_Socket_LongPads
Connections:
- net /BUSAK: no longer U33.11 (I0b)
- net CPU_Q: now also U5.3
- net R/W: no longer U30.8 (I3a)
- net at U5.1: now also U33.2 (I0a)
- net /BUSRQ: no longer names the net of U32.33 (~{DMA/BREQ})
- net /BUSRQ: no longer U33.7 (O1b)
- net /SO: no longer names the net of RR2.4 (R3)
- net B_/BUSAK: no longer names the net of U33.9 (O0b)
- net B_/BUSRQ: no longer names the net of U33.13 (I1b)
- net B_DT/R: no longer names the net of U30.12 (O3a)
- no-connect marks 15 -> 23
Other:
- note removed: "1-2 6802 2-3 6809 / 6502"
- note removed: "1-2 6809 3-4 6502 5-6 6502 alternate"
- company: N8VEM Users Group -> (none)
- title: 6809 and 6502 ATX and 6U -> 6809PC

Commit message: PCB in progress
Parts:
- C58: footprint Capacitor_THT:C_Disc_D5.0mm_W2.5mm_P5.00mm -> Custom:STD_DDW_CAP
- JP2: value JUMPER -> CPU XTAL; footprint Connector_PinHeader_2.54mm:PinHeader_1x02_P2.54mm_Vertical -> Custom:STD_DDW_PINHEAD_V_1x02
- K2: footprint Connector_PinHeader_2.54mm:PinHeader_1x03_P2.54mm_Vertical -> Custom:STD_DDW_PINHEAD_V_1x03
- P14: renamed from P10; footprint Package_DIP:DIP-14_W7.62mm_Socket_LongPads -> Custom:STD_DDW_DIP14
- P15: renamed from P11; value CONN_4X2 -> CPU CLOCK SPEED; footprint Connector_PinHeader_2.54mm:PinHeader_2x04_P2.54mm_Vertical -> Custom:STD_DDW_PINHEAD_V_2x04
- RR2: footprint Resistor_THT:R_Array_SIP10 -> Custom:STD_DDW_SIP10
- U1, U17, U18, U21, U5, U6: footprint Package_DIP:DIP-14_W7.62mm_Socket_LongPads -> Custom:STD_DDW_DIP14
- U30: renamed from U29; footprint Package_DIP:DIP-16_W7.62mm_Socket_LongPads -> Custom:STD_DDW_DIP16
- U31: renamed from U30; footprint Package_DIP:DIP-20_W7.62mm_Socket_LongPads -> Custom:STD_DDW_DIP20
- U32: renamed from U31; footprint Package_DIP:DIP-20_W7.62mm_Socket_LongPads -> Custom:STD_DDW_DIP20
- U33: renamed from U32; footprint Package_DIP:DIP-40_W15.24mm_Socket_LongPads -> Custom:STD_DDW_DIP40
- U34: renamed from U33; footprint Package_DIP:DIP-20_W7.62mm_Socket_LongPads -> Custom:STD_DDW_DIP20

Commit message: V1.1
Parts:
- removed JP2: CPU XTAL, Custom:STD_DDW_PINHEAD_V_1x02, symbol Jumper:Jumper_2_Open
Connections:
- net GND: now also U33.39 (XTAL)
- net DMA: now reaches RR2.4 (R3)
- net DMA: now also U33.33 (~{DMA/BREQ})
- no-connect marks 23 -> 21
Changed lines of the file:
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@@
 	)
 	(no_connect
-		(at 247.65 90.17)
-	)
-	(no_connect
-		(at 383.54 66.04)
-	)
-	(no_connect
 		(at 106.68 228.6)
 	)
@@
 	(wire
 		(pts
-			(xy 186.69 102.87) (xy 200.66 102.87)
+			(xy 186.69 102.87) (xy 247.65 102.87)
 		)
 		(stroke
@@
 	(wire
 		(pts
+			(xy 382.27 66.04) (xy 383.54 66.04)
+		)
+		(stroke
+			(width 0)
+			(type default)
+		)
+	)
+	(wire
+		(pts
 			(xy 273.05 90.17) (xy 284.48 90.17)
 		)
@@
 	(wire
 		(pts
-			(xy 210.82 102.87) (xy 247.65 102.87)
-		)
-		(stroke
-			(width 0)
-			(type default)
-		)
-	)
-	(wire
-		(pts
 			(xy 255.27 241.3) (xy 252.73 241.3)
 		)
@@
 	(wire
 		(pts
+			(xy 215.9 90.17) (xy 247.65 90.17)
+		)
+		(stroke
+			(width 0)
+			(type default)
+		)
+	)
+	(wire
+		(pts
 			(xy 393.7 60.96) (xy 394.97 60.96)
 		)
@@
 		)
 	)
+	(global_label "DMA"
+		(shape input)
+		(at 382.27 66.04 180)
+		(fields_autoplaced yes)
+		(effects
+			(font
+				(size 1.27 1.27)
+			)
+			(justify right)
+		)
+		(property "Intersheetrefs" "${INTERSHEET_REFS}"
+			(at 376.129 66.04 0)
+			(effects
+				(font
+					(size 1.27 1.27)
+				)
+				(justify right)
+				(hide yes)
+			)
+		)
+	)
 	(global_label "LA13"
 		(shape input)
@@
 		)
 	)
+	(global_label "DMA"
+		(shape input)
+		(at 215.9 90.17 180)
+		(fields_autoplaced yes)
+		(effects
+			(font
+				(size 1.27 1.27)
+			)
+			(justify right)
+		)
+		(property "Intersheetrefs" "${INTERSHEET_REFS}"
+			(at 209.759 90.17 0)
+			(effects
+				(font
+					(size 1.27 1.27)
+				)
+				(justify right)
+				(hide yes)
+			)
+		)
+	)
 	(symbol
 		(lib_id "Device:R_Network09")
@@
 		)
 		(property "Value" "CPU CLOCK SPEED"
-			(at 125.73 68.58 90)
+			(at 129.032 76.708 0)
 			(effects
 				(font
@@
 				)
 			)
-		)
-	)
-	(symbol
-		(lib_id "Jumper:Jumper_2_Open")
-		(at 205.74 102.87 0)
-		(unit 1)
-		(exclude_from_sim yes)
-		(in_bom yes)
-		(on_board yes)
-		(dnp no)
-		(property "Reference" "JP2"
-			(at 205.74 99.06 0)
-			(effects
-				(font
-					(size 1.524 1.524)
-				)
-			)
-		)
-		(property "Value" "CPU XTAL"
-			(at 205.74 104.902 0)
-			(effects
-				(font
-					(size 1.016 1.016)
-				)
-			)
-		)
-		(property "Footprint" "Custom:STD_DDW_PINHEAD_V_1x02"
-			(at 205.74 102.87 0)
-			(effects
-				(font
-					(size 1.27 1.27)
-				)
-				(hide yes)
-			)
-		)
-		(property "Datasheet" "~"
-			(at 205.74 102.87 0)
-			(effects
-				(font
-					(size 1.27 1.27)
-				)
-				(hide yes)
-			)
-		)
-		(property "Description" "Jumper, 2-pole, open"
-			(at 205.74 102.87 0)
-			(effects
-				(font
-					(size 1.27 1.27)
-				)
-				(hide yes)
-			)
-		)
-		(pin "1"
-		)
-		(pin "2"
-		)
-		(instances
-			(project "6x0x-6U"
-				(path "/d94f9d60-5ece-4752-b49c-b0d1c95f35bc/00000000-0000-0000-0000-0000526c8e8e"
-					(reference "JP2")
-					(unit 1)
-				)
-			)

Commit message: 6809PC work
Parts:
- K2: value CONN_3 -> MMU-INTA
Changed lines of the file:
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@@
 	(title_block
 		(title "6809PC")
-		(date "2025-01-21")
-		(rev "001")
+		(date "2025-05-17")
+		(rev "002")
 		(comment 1 "https://github.com/danwerner21/6809PC")
 		(comment 2 "Based on work by Andrew Lynch and John Coffman")
@@
 			)
 		)
-		(property "Value" "CONN_3"
+		(property "Value" "MMU-INTA"
 			(at 299.72 144.78 90)
 			(effects

Commit message: fix issue with ISA RW select lines
Parts:
- added unit 1 of U17
Connections:
- net CPU_Q: now also U17.1
- net /IORQ: no longer names the net of U34.15 (I2b)
- net /IORQ: now also U17.2
- net B_/IORQ renamed BUSALE
Other:
- note added: "Bus Address Latch Enable. The address bus is latched on the rising edge of this signal."
- note removed: "similar to /MREQ"
Changed lines of the file:
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@@
 	(wire
 		(pts
-			(xy 328.93 182.88) (xy 341.63 182.88)
-		)
-		(stroke
-			(width 0)
-			(type default)
-		)
-	)
-	(wire
-		(pts
 			(xy 194.31 222.25) (xy 194.31 241.3)
 		)
@@
 	(wire
 		(pts
+			(xy 257.81 195.58) (xy 257.81 182.88)
+		)
+		(stroke
+			(width 0)
+			(type default)
+		)
+	)
+	(wire
+		(pts
 			(xy 217.17 222.25) (xy 217.17 226.06)
 		)
@@
 	(wire
 		(pts
+			(xy 328.93 182.88) (xy 346.71 182.88)
+		)
+		(stroke
+			(width 0)
+			(type default)
+		)
+	)
+	(wire
+		(pts
 			(xy 171.45 73.66) (xy 189.23 73.66)
 		)
@@
 	(wire
 		(pts
-			(xy 303.53 182.88) (xy 300.99 182.88)
+			(xy 151.13 223.52) (xy 154.94 223.52)
 		)
 		(stroke
@@
 	(wire
 		(pts
-			(xy 151.13 223.52) (xy 154.94 223.52)
+			(xy 257.81 182.88) (xy 303.53 182.88)
 		)
 		(stroke
@@
 	(wire
 		(pts
+			(xy 238.76 195.58) (xy 242.57 195.58)
+		)
+		(stroke
+			(width 0)
+			(type default)
+		)
+	)
+	(wire
+		(pts
 			(xy 133.35 73.66) (xy 171.45 73.66)
 		)
@@
 		)
 	)
-	(text "similar to /MREQ"
+	(text "Bus Address Latch Enable. The address bus is latched on the rising edge of this signal."
 		(exclude_from_sim no)
-		(at 350.52 168.91 0)
+		(at 243.078 201.422 0)
 		(effects
 			(font
-				(size 1.524 1.524)
+				(size 1.27 1.27)
 			)
-			(justify left bottom)
 		)
 	)
@@
 		)
 	)
-	(global_label "mD4"
-		(shape bidirectional)
-		(at 255.27 236.22 0)
+	(global_label "CPU_Q"
+		(shape input)
+		(at 238.76 195.58 180)
 		(effects
 			(font
 				(size 1.524 1.524)
 			)
-			(justify left)
+			(justify right)
 		)
 		(property "Intersheetrefs" "${INTERSHEET_REFS}"
-			(at 255.27 236.22 0)
+			(at 238.76 195.58 0)
 			(effects
 				(font
@@
 		)
 	)
-	(global_label "/HALT"
-		(shape input)
-		(at 236.22 92.71 180)
+	(global_label "mD4"
+		(shape bidirectional)
+		(at 255.27 236.22 0)
 		(effects
 			(font
 				(size 1.524 1.524)
 			)
-			(justify right)
+			(justify left)
 		)
 		(property "Intersheetrefs" "${INTERSHEET_REFS}"
-			(at 236.22 92.71 0)
+			(at 255.27 236.22 0)
 			(effects
 				(font
@@
 		)
 	)
-	(global_label "/IORQ"
+	(global_label "/HALT"
 		(shape input)
-		(at 300.99 182.88 180)
+		(at 236.22 92.71 180)
 		(effects
 			(font
@@
 		)
 		(property "Intersheetrefs" "${INTERSHEET_REFS}"
-			(at 300.99 182.88 0)
+			(at 236.22 92.71 0)
 			(effects
 				(font
@@
 		)
 	)
-	(global_label "B_/IORQ"
-		(shape output)
-		(at 341.63 182.88 0)
-		(effects
-			(font
-				(size 1.524 1.524)
-			)
-			(justify left)
-		)
-		(property "Intersheetrefs" "${INTERSHEET_REFS}"
-			(at 341.63 182.88 0)
-			(effects
-				(font
-					(size 1.27 1.27)
-				)
-				(hide yes)
-			)
-		)
-	)
 	(global_label "mD7"
 		(shape bidirectional)
@@
 		)
 	)
+	(global_label "BUSALE"
+		(shape output)
+		(at 346.71 182.88 0)
+		(fields_autoplaced yes)
+		(effects
+			(font
+				(size 1.27 1.27)
+			)
+			(justify left)
+		)
+		(property "Intersheetrefs" "${INTERSHEET_REFS}"
+			(at 356.1167 182.88 0)
+			(effects
+				(font
+					(size 1.27 1.27)
+				)
+				(justify left)
+				(hide yes)
+			)
+		)
+	)
 	(global_label "B_/INT"
 		(shape input)
@@
 					(unit 1)
 				)
+			)
+		)
+	)
+	(symbol
+		(lib_id "74xx:74LS14")
+		(at 250.19 195.58 0)
+		(unit 1)
+		(exclude_from_sim no)
+		(in_bom yes)
+		(on_board yes)
+		(dnp no)
+		(property "Reference" "U17"
+			(at 254 193.04 0)
+			(effects
+				(font
+					(size 1.016 1.016)
+				)
+			)
+		)
+		(property "Value" "74LS14"
+			(at 255.27 198.12 0)
+			(effects
+				(font
+					(size 1.016 1.016)
+				)
+			)
+		)
+		(property "Footprint" "Custom:STD_DDW_DIP14"
+			(at 250.19 195.58 0)
+			(effects
+				(font
+					(size 1.27 1.27)
+				)
+				(hide yes)
+			)
+		)
+		(property "Datasheet" "http://www.ti.com/lit/gpn/sn74LS14"
+			(at 250.19 195.58 0)
+			(effects
+				(font
+					(size 1.27 1.27)
+				)
+				(hide yes)
+			)
+		)
+		(property "Description" "Hex inverter schmitt trigger"
+			(at 250.19 195.58 0)
+			(effects
+				(font
+					(size 1.27 1.27)
+				)
+				(hide yes)
+			)
+		)
+		(pin "14"
+		)
+		(pin "7"
+		)
+		(pin "1"
+		)
+		(pin "8"
+		)
+		(pin "6"
+		)
+		(pin "9"
+		)
+		(pin "4"
+		)
+		(pin "3"
+		)
+		(pin "10"
+		)
+		(pin "2"
+		)
+		(pin "12"
+		)
+		(pin "13"
+		)
+		(pin "5"
+		)
+		(pin "11"
+		)
+		(instances
+			(project "6809PC-6U"
+				(path "/d94f9d60-5ece-4752-b49c-b0d1c95f35bc/00000000-0000-0000-0000-0000526c8e8e"
+					(reference "U17")
+					(unit 1)
+				)

Commit message: fix bus issue
Connections:
- net CLK: no longer U31.2 (I0a)
- net CPU_E: now also U31.2 (I0a)
Changed lines of the file:
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@@
 	(title_block
 		(title "6809PC")
-		(date "2025-05-17")
-		(rev "002")
+		(date "2025-05-31")
+		(rev "003")
 		(comment 1 "https://github.com/danwerner21/6809PC")
 		(comment 2 "Based on work by Andrew Lynch and John Coffman")
@@
 		)
 	)
-	(global_label "CLK"
-		(shape input)
-		(at 78.74 220.98 180)
-		(effects
-			(font
-				(size 1.524 1.524)
-			)
-			(justify right)
-		)
-		(property "Intersheetrefs" "${INTERSHEET_REFS}"
-			(at 78.74 220.98 0)
-			(effects
-				(font
-					(size 1.27 1.27)
-				)
-				(hide yes)
-			)
-		)
-	)
 	(global_label "CPU_Q"
 		(shape input)
@@
 			(effects
 				(font
+					(size 1.27 1.27)
+				)
+				(hide yes)
+			)
+		)
+	)
+	(global_label "CPU_E"
+		(shape input)
+		(at 78.74 220.98 180)
+		(effects
+			(font
+				(size 1.524 1.524)
+			)
+			(justify right)
+		)
+		(property "Intersheetrefs" "${INTERSHEET_REFS}"
+			(at 78.74 220.98 0)
+			(effects
+				(font
