File: ECBbus.kicad_sch (KiCad schematic)
At the start: 12 parts, among them J1 IRQ Selection, J10 Bus_ISA_8bit, J13 IRQ Selection, J14 Bus_ISA_8bit, J2 IRQ Selection, J3 Bus_ISA_8bit, J4 Bus_ISA_8bit, J5 IRQ Selection, J6 Bus_ISA_8bit, J7 IRQ Selection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

Commit message: isa work
Connections:
- net /RESET renamed RESET
Changed lines of the file:
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@@
 		)
 	)
-	(global_label "{slash}RESET"
-		(shape input)
-		(at 60.96 124.46 180)
-		(effects
-			(font
-				(size 1.524 1.524)
-			)
-			(justify right)
-		)
-		(property "Intersheetrefs" "${INTERSHEET_REFS}"
-			(at 60.96 124.46 0)
-			(effects
-				(font
-					(size 1.27 1.27)
-				)
-				(hide yes)
-			)
-		)
-	)
 	(global_label "B_SMEMR"
 		(shape output)
@@
 		)
 	)
-	(global_label "{slash}RESET"
-		(shape input)
-		(at 156.21 26.67 180)
-		(effects
-			(font
-				(size 1.524 1.524)
-			)
-			(justify right)
-		)
-		(property "Intersheetrefs" "${INTERSHEET_REFS}"
-			(at 156.21 26.67 0)
-			(effects
-				(font
-					(size 1.27 1.27)
-				)
-				(hide yes)
-			)
-		)
-	)
 	(global_label "B_D4"
 		(shape bidirectional)
@@
 		)
 	)
-	(global_label "{slash}RESET"
-		(shape input)
-		(at 156.21 124.46 180)
-		(effects
-			(font
-				(size 1.524 1.524)
-			)
-			(justify right)
-		)
-		(property "Intersheetrefs" "${INTERSHEET_REFS}"
-			(at 156.21 124.46 0)
-			(effects
-				(font
-					(size 1.27 1.27)
-				)
-				(hide yes)
-			)
-		)
-	)
 	(global_label "BUSCLK"
 		(shape input)
@@
 		)
 	)
-	(global_label "{slash}RESET"
-		(shape input)
-		(at 347.98 25.4 180)
-		(effects
-			(font
-				(size 1.524 1.524)
-			)
-			(justify right)
-		)
-		(property "Intersheetrefs" "${INTERSHEET_REFS}"
-			(at 347.98 25.4 0)
-			(effects
-				(font
-					(size 1.27 1.27)
-				)
-				(hide yes)
-			)
-		)
-	)
 	(global_label "B_D4"
 		(shape bidirectional)
@@
 		)
 	)
+	(global_label "RESET"
+		(shape input)
+		(at 156.21 26.67 180)
+		(effects
+			(font
+				(size 1.524 1.524)
+			)
+			(justify right)
+		)
+		(property "Intersheetrefs" "${INTERSHEET_REFS}"
+			(at 156.21 26.67 0)
+			(effects
+				(font
+					(size 1.27 1.27)
+				)
+				(hide yes)
+			)
+		)
+	)
 	(global_label "TC"
 		(shape input)
@@
 		)
 	)
-	(global_label "{slash}RESET"
-		(shape input)
-		(at 251.46 25.4 180)
-		(effects
-			(font
-				(size 1.524 1.524)
-			)
-			(justify right)
-		)
-		(property "Intersheetrefs" "${INTERSHEET_REFS}"
-			(at 251.46 25.4 0)
-			(effects
-				(font
-					(size 1.27 1.27)
-				)
-				(hide yes)
-			)
-		)
-	)
 	(global_label "B_A8"
 		(shape bidirectional)
@@
 		)
 	)
-	(global_label "{slash}RESET"
-		(shape input)
-		(at 62.23 27.94 180)
-		(effects
-			(font
-				(size 1.524 1.524)
-			)
-			(justify right)
-		)
-		(property "Intersheetrefs" "${INTERSHEET_REFS}"
-			(at 62.23 27.94 0)
-			(effects
-				(font
-					(size 1.27 1.27)
-				)
-				(hide yes)
-			)
-		)
-	)
 	(global_label "isa_iq_1"
 		(shape input)
@@
 		)
 	)
+	(global_label "RESET"
+		(shape input)
+		(at 60.96 124.46 180)
+		(effects
+			(font
+				(size 1.524 1.524)
+			)
+			(justify right)
+		)
+		(property "Intersheetrefs" "${INTERSHEET_REFS}"
+			(at 60.96 124.46 0)
+			(effects
+				(font
+					(size 1.27 1.27)
+				)
+				(hide yes)
+			)
+		)
+	)
 	(global_label "isa_iq_3"
 		(shape input)
@@
 		)
 	)
+	(global_label "RESET"
+		(shape input)
+		(at 347.98 25.4 180)
+		(effects
+			(font
+				(size 1.524 1.524)
+			)
+			(justify right)
+		)
+		(property "Intersheetrefs" "${INTERSHEET_REFS}"
+			(at 347.98 25.4 0)
+			(effects
+				(font
+					(size 1.27 1.27)
+				)
+				(hide yes)
+			)
+		)
+	)
 	(global_label "B_D1"
 		(shape bidirectional)
@@
 		)
 	)
+	(global_label "RESET"
+		(shape input)
+		(at 156.21 124.46 180)
+		(effects
+			(font
+				(size 1.524 1.524)
+			)
+			(justify right)
+		)
+		(property "Intersheetrefs" "${INTERSHEET_REFS}"
+			(at 156.21 124.46 0)
+			(effects
+				(font
+					(size 1.27 1.27)
+				)
+				(hide yes)
+			)
+		)
+	)
 	(global_label "isa_iq_5"
 		(shape input)
@@
 		)
 	)
+	(global_label "RESET"
+		(shape input)
+		(at 62.23 27.94 180)
+		(effects
+			(font
+				(size 1.524 1.524)
+			)
+			(justify right)
+		)
+		(property "Intersheetrefs" "${INTERSHEET_REFS}"
+			(at 62.23 27.94 0)
+			(effects
+				(font
+					(size 1.27 1.27)
+				)
+				(hide yes)
+			)
+		)
+	)
 	(global_label "B_A2"
 		(shape bidirectional)
@@
 				(hide yes)
 			)
+		)
+	)
+	(global_label "RESET"
+		(shape input)
+		(at 251.46 25.4 180)
+		(effects
+			(font
+				(size 1.524 1.524)
+			)
+			(justify right)
+		)
+		(property "Intersheetrefs" "${INTERSHEET_REFS}"
+			(at 251.46 25.4 0)
+			(effects
+				(font
+					(size 1.27 1.27)
+				)
+				(hide yes)
+			)
