File: Reset.kicad_sch (KiCad schematic)
At the start: 4 parts, among them SW2 MOM CNCT, U23 DS1233

Commit message: Schematic in progress
Parts:
- C57: renamed from C56; footprint C2 -> Capacitor_THT:C_Disc_D5.0mm_W2.5mm_P5.00mm
- JP1: footprint PIN_ARRAY_2X1 -> Connector_PinHeader_2.54mm:PinHeader_1x02_P2.54mm_Vertical
- SW2: footprint SW_PUSH_SMALL -> Button_Switch_THT:SW_Tactile_Straight_KSL0Axx1LFTR
- renumbered U23 to U28
Other:
- company: N8VEM Users Group -> (none)
- title: 6809 and 6502 ATX and 6U -> 6809PC
Changed lines of the file:
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@@
 	(paper "A")
 	(title_block
-		(title "6809 and 6502 ATX and 6U")
-		(date "19 feb 2014")
-		(rev "012")
-		(company "N8VEM Users Group")
-		(comment 1 "Licensed for hobbyist use only.  All other rights reserved.")
-		(comment 2 "Copyright (c) 2013-2014  Andrew Lynch and John Coffman")
+		(title "6809PC")
+		(date "2025-01-21")
+		(rev "001")
+		(comment 1 "https://github.com/danwerner21/6809PC")
+		(comment 2 "Based on work by Andrew Lynch and John Coffman")
 	)
 	(junction
@@
 			)
 		)
-		(property "Footprint" "PIN_ARRAY_2X1"
+		(property "Footprint" "Connector_PinHeader_2.54mm:PinHeader_1x02_P2.54mm_Vertical"
 			(at 133.35 100.33 0)
 			(effects
@@
 			)
 		)
-		(property "Footprint" "SW_PUSH_SMALL"
+		(property "Footprint" "Button_Switch_THT:SW_Tactile_Straight_KSL0Axx1LFTR"
 			(at 110.49 104.14 0)
 			(effects
@@
 		(on_board yes)
 		(dnp no)
-		(property "Reference" "C56"
+		(property "Reference" "C57"
 			(at 101.092 101.6 0)
 			(effects
@@
 			)
 		)
-		(property "Footprint" "C2"
+		(property "Footprint" "Capacitor_THT:C_Disc_D5.0mm_W2.5mm_P5.00mm"
 			(at 107.6452 107.95 0)
 			(effects
@@
 			(project "6809PC-6U"
 				(path "/d94f9d60-5ece-4752-b49c-b0d1c95f35bc/00000000-0000-0000-0000-0000526d81d3"
-					(reference "C56")
+					(reference "C57")
 					(unit 1)
 				)
@@
 		(on_board yes)
 		(dnp no)
-		(property "Reference" "#PWR052"
+		(property "Reference" "#PWR064"
 			(at 100.33 87.63 0)
 			(effects
@@
 			(project "6809PC-6U"
 				(path "/d94f9d60-5ece-4752-b49c-b0d1c95f35bc/00000000-0000-0000-0000-0000526d81d3"
-					(reference "#PWR052")
+					(reference "#PWR064")
 					(unit 1)
 				)
@@
 		(on_board yes)
 		(dnp no)
-		(property "Reference" "U23"
+		(property "Reference" "U28"
 			(at 96.52 72.39 90)
 			(effects
@@
 			(project "6809PC-6U"
 				(path "/d94f9d60-5ece-4752-b49c-b0d1c95f35bc/00000000-0000-0000-0000-0000526d81d3"
-					(reference "U23")
+					(reference "U28")
 					(unit 1)
 				)
@@
 		(on_board yes)
 		(dnp no)
-		(property "Reference" "#PWR054"
+		(property "Reference" "#PWR066"
 			(at 123.19 119.38 0)
 			(effects
@@
 			(project "6809PC-6U"
 				(path "/d94f9d60-5ece-4752-b49c-b0d1c95f35bc/00000000-0000-0000-0000-0000526d81d3"
-					(reference "#PWR054")
+					(reference "#PWR066")
 					(unit 1)
 				)
@@
 		(on_board yes)
 		(dnp no)
-		(property "Reference" "#PWR053"
+		(property "Reference" "#PWR065"
 			(at 107.95 85.09 0)
 			(effects
@@
 			(project "6809PC-6U"
 				(path "/d94f9d60-5ece-4752-b49c-b0d1c95f35bc/00000000-0000-0000-0000-0000526d81d3"
-					(reference "#PWR053")
+					(reference "#PWR065")
 					(unit 1)
 				)

Commit message: PCB in progress
Parts:
- C57: footprint Capacitor_THT:C_Disc_D5.0mm_W2.5mm_P5.00mm -> Custom:STD_DDW_CAP
- JP1: footprint Connector_PinHeader_2.54mm:PinHeader_1x02_P2.54mm_Vertical -> Custom:STD_DDW_PINHEAD_V_1x02
- SW2: footprint Button_Switch_THT:SW_Tactile_Straight_KSL0Axx1LFTR -> Custom:STD_DDW_TACTSW
- U29: renamed from U28; footprint Package_TO_SOT_THT:TO-92L_HandSolder -> Custom:STD_DDW_TO92
Changed lines of the file:
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@@
 			)
 		)
-		(property "Footprint" "Connector_PinHeader_2.54mm:PinHeader_1x02_P2.54mm_Vertical"
+		(property "Footprint" "Custom:STD_DDW_PINHEAD_V_1x02"
 			(at 133.35 100.33 0)
 			(effects
@@
 			)
 		)
-		(property "Footprint" "Button_Switch_THT:SW_Tactile_Straight_KSL0Axx1LFTR"
+		(property "Footprint" "Custom:STD_DDW_TACTSW"
 			(at 110.49 104.14 0)
 			(effects
@@
 			)
 		)
-		(property "Footprint" "Capacitor_THT:C_Disc_D5.0mm_W2.5mm_P5.00mm"
+		(property "Footprint" "Custom:STD_DDW_CAP"
 			(at 107.6452 107.95 0)
 			(effects
@@
 		(on_board yes)
 		(dnp no)
-		(property "Reference" "#PWR064"
+		(property "Reference" "#PWR0102"
 			(at 100.33 87.63 0)
 			(effects
@@
 			(project "6809PC-6U"
 				(path "/d94f9d60-5ece-4752-b49c-b0d1c95f35bc/00000000-0000-0000-0000-0000526d81d3"
-					(reference "#PWR064")
+					(reference "#PWR0102")
 					(unit 1)
 				)
@@
 		(on_board yes)
 		(dnp no)
-		(property "Reference" "U28"
+		(property "Reference" "U29"
 			(at 96.52 72.39 90)
 			(effects
@@
 			)
 		)
-		(property "Footprint" "Package_TO_SOT_THT:TO-92L_HandSolder"
+		(property "Footprint" "Custom:STD_DDW_TO92"
 			(at 102.87 72.39 0)
 			(effects
@@
 			(project "6809PC-6U"
 				(path "/d94f9d60-5ece-4752-b49c-b0d1c95f35bc/00000000-0000-0000-0000-0000526d81d3"
-					(reference "U28")
+					(reference "U29")
 					(unit 1)
 				)
@@
 		(on_board yes)
 		(dnp no)
-		(property "Reference" "#PWR066"
+		(property "Reference" "#PWR0104"
 			(at 123.19 119.38 0)
 			(effects
@@
 			(project "6809PC-6U"
 				(path "/d94f9d60-5ece-4752-b49c-b0d1c95f35bc/00000000-0000-0000-0000-0000526d81d3"
-					(reference "#PWR066")
+					(reference "#PWR0104")
 					(unit 1)
 				)
@@
 		(on_board yes)
 		(dnp no)
-		(property "Reference" "#PWR065"
+		(property "Reference" "#PWR0103"
 			(at 107.95 85.09 0)
 			(effects
@@
 			(project "6809PC-6U"
 				(path "/d94f9d60-5ece-4752-b49c-b0d1c95f35bc/00000000-0000-0000-0000-0000526d81d3"
-					(reference "#PWR065")
-					(unit 1)
-				)
+					(reference "#PWR0103")
+					(unit 1)
+				)

Commit message: 6809PC work
Parts:
- SW2: value MOM CNCT -> RESET
Changed lines of the file:
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@@
 	(title_block
 		(title "6809PC")
-		(date "2025-01-21")
-		(rev "001")
+		(date "2025-05-17")
+		(rev "002")
 		(comment 1 "https://github.com/danwerner21/6809PC")
 		(comment 2 "Based on work by Andrew Lynch and John Coffman")
@@
 			)
 		)
-		(property "Value" "MOM CNCT"
+		(property "Value" "RESET"
 			(at 117.602 104.14 0)
 			(effects

Commit message: isa work
Parts:
- added U17: 74LS14, Custom:STD_DDW_DIP14, symbol 74xx:74LS14
Connections:
- net /RESET: now also U17.9
- new net RESET: U17.8
Changed lines of the file:
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@@
+	)
+	(junction
+		(at 133.35 91.44)
+		(diameter 0)
+		(color 0 0 0 0)
 	)
 	(junction
@@
 	(wire
 		(pts
+			(xy 148.59 82.55) (xy 153.67 82.55)
+		)
+		(stroke
+			(width 0)
+			(type default)
+		)
+	)
+	(wire
+		(pts
 			(xy 115.57 111.76) (xy 123.19 111.76)
 		)
@@
 	(wire
 		(pts
+			(xy 133.35 91.44) (xy 135.89 91.44)
+		)
+		(stroke
+			(width 0)
+			(type default)
+		)
+	)
+	(wire
+		(pts
 			(xy 105.41 77.47) (xy 105.41 87.63)
 		)
@@
 	(wire
 		(pts
+			(xy 133.35 82.55) (xy 133.35 91.44)
+		)
+		(stroke
+			(width 0)
+			(type default)
+		)
+	)
+	(wire
+		(pts
 			(xy 106.68 111.76) (xy 115.57 111.76)
 		)
@@
 	(wire
 		(pts
-			(xy 128.27 91.44) (xy 135.89 91.44)
+			(xy 128.27 91.44) (xy 133.35 91.44)
 		)
 		(stroke
@@
 			)
 			(justify right bottom)
+		)
+	)
+	(global_label "RESET"
+		(shape output)
+		(at 153.67 82.55 0)
+		(effects
+			(font
+				(size 1.524 1.524)
+			)
+			(justify left)
+		)
+		(property "Intersheetrefs" "${INTERSHEET_REFS}"
+			(at 153.67 82.55 0)
+			(effects
+				(font
+					(size 1.27 1.27)
+				)
+				(hide yes)
+			)
 		)
 	)
@@
 				)
 			)
+		)
+	)
+	(symbol
+		(lib_id "74xx:74LS14")
+		(at 140.97 82.55 0)
+		(unit 4)
+		(exclude_from_sim no)
+		(in_bom yes)
+		(on_board yes)
+		(dnp no)
+		(property "Reference" "U17"
+			(at 145.923 79.629 0)
+			(effects
+				(font
+					(size 1.524 1.524)
+				)
+			)
+		)
+		(property "Value" "74LS14"
+			(at 145.796 85.725 0)
+			(effects
+				(font
+					(size 1.524 1.524)
+				)
+			)
+		)
+		(property "Footprint" "Custom:STD_DDW_DIP14"
+			(at 140.97 82.55 0)
+			(effects
+				(font
+					(size 1.27 1.27)
+				)
+				(hide yes)
+			)
+		)
+		(property "Datasheet" "http://www.ti.com/lit/gpn/sn74LS14"
+			(at 140.97 82.55 0)
+			(effects
+				(font
+					(size 1.27 1.27)
+				)
+				(hide yes)
+			)
+		)
+		(property "Description" "Hex inverter schmitt trigger"
+			(at 140.97 82.55 0)
+			(effects
+				(font
+					(size 1.27 1.27)
+				)
+				(hide yes)
+			)
+		)
+		(pin "2"
+		)
+		(pin "8"
+		)
+		(pin "7"
+		)
+		(pin "9"
+		)
+		(pin "14"
+		)
+		(pin "1"
+		)
+		(pin "4"
+		)
+		(pin "3"
+		)
+		(pin "6"
+		)
+		(pin "5"
+		)
+		(pin "12"
+		)
+		(pin "13"
+		)
+		(pin "11"
+		)
+		(pin "10"
+		)
+		(instances
+			(project "6809PC-6U"
+				(path "/d94f9d60-5ece-4752-b49c-b0d1c95f35bc/00000000-0000-0000-0000-0000526d81d3"
+					(reference "U17")
+					(unit 4)
+				)
+			)
